File: t100-dcmotor/t100-dcmotor.kicad_pcb (KiCad board)
At the start: 2 copper layers, 34.5 x 99.5 mm, 27 parts, among them J1 T100-IN, J2 T100-OUT, J3 Motor, U1 ATSAMD11D14A-SS, U2 VNH7070BAS, X1 SWD

Commit message: WIP
Parts:
- removed JP1: F1, Jumper:SolderJumper-3_P2.0mm_Open_TrianglePad1.0x1.5mm
- removed JP2: F2, Jumper:SolderJumper-3_P2.0mm_Open_TrianglePad1.0x1.5mm
- added R12: A-270R B-N/A Z-10k, Resistor_SMD:R_0805_2012Metric_Pad1.15x1.40mm_HandSolder, F.Cu at (104.0, 67.0)
- added R13: A-N/A B-270R Z-10k, Resistor_SMD:R_0805_2012Metric_Pad1.15x1.40mm_HandSolder, F.Cu at (104.0, 63.0)
- added R14: 10k, Resistor_SMD:R_0805_2012Metric_Pad1.15x1.40mm_HandSolder, F.Cu at (94.0, 74.5)
- added R15: 10k, Resistor_SMD:R_0805_2012Metric_Pad1.15x1.40mm_HandSolder, F.Cu at (94.0, 71.0)
- J3: value Motor -> Conn_01x08_Female; footprint device.farm:DG142R-6-5.08 -> device.farm:DG235-3.81-08P
- R7, R8: value 1k -> 10k
- moved J3 5.00 mm to (87.5, 124.5)
Connections:
- U1 pad 19: Net-(U1-Pad19) -> /ADDR
- U1 pad 4: /FNC1 -> /STOP_1
- U1 pad 5: /FNC2 -> /STOP_2
Routing:
- net /STOP_1: track 0.00 -> 117.5 mm, vias 0 -> 1
- net /STOP_2: track 0.00 -> 115.3 mm, vias 0 -> 1
- net GND: track 148.8 -> 115.1 mm, vias 19 -> 31
- net /ADDR: track 0.00 -> 28.2 mm
- net /FNC2: track 24.5 -> 0.00 mm
- net /FNC1: track 20.3 -> 0.00 mm
- net Net-(J3-Pad3): track 41.0 -> 32.2 mm
- net Net-(FB1-Pad1): track 49.9 -> 42.8 mm
- net Net-(J3-Pad4): track 44.0 -> 38.8 mm
- net +3V3: track 154.7 -> 159.2 mm
- net +12V: track 105.4 -> 107.4 mm
- net /MOTOR_M: track 29.1 -> 28.1 mm
- net +5V: track 48.0 -> 48.6 mm
- added copper zone on F.Cu, net GND
Other:
- board text added: "12V DC MOTOR DRIVER W/ HALL ENCODER"
- board text added: "5V"
- board text added: "AXIS"
- board text added: "GND"
- board text added: "ST1"
- board text added: "ST2"
- board text removed: "12V DC MOTOR DRIVER WITH ENCODER"
- board text removed: "A"
- board text removed: "B"
- board text removed: "C"
- board text removed: "D"
- board text removed: "HS+"
- board text removed: "HS-"
