File: t100-dcmotor/t100-dcmotor.sch (KiCad schematic (older format))
At the start: 27 parts, among them J1 T100-IN, J2 T100-OUT, J3 Motor, U1 ATSAMD11D14A-SS, U2 VNH7070BAS, X1 SWD

Commit message: WIP
Parts:
- removed J3: Motor, device.farm:DG142R-6-5.08, symbol Connector:Conn_01x06_Female
- removed JP1: F1, Jumper:SolderJumper-3_P2.0mm_Open_TrianglePad1.0x1.5mm, symbol Jumper:SolderJumper_3_Open
- removed JP2: F2, Jumper:SolderJumper-3_P2.0mm_Open_TrianglePad1.0x1.5mm, symbol Jumper:SolderJumper_3_Open
- added J3: Conn_01x08_Female, device.farm:DG235-3.81-08P, symbol Connector:Conn_01x08_Female
- added R12: A-270R B-N/A Z-10k, Resistor_SMD:R_0805_2012Metric_Pad1.15x1.40mm_HandSolder, symbol Device:R
- added R13: A-N/A B-270R Z-10k, Resistor_SMD:R_0805_2012Metric_Pad1.15x1.40mm_HandSolder, symbol Device:R
- added R14, R15: 10k, Resistor_SMD:R_0805_2012Metric_Pad1.15x1.40mm_HandSolder, symbol Device:R
- R7, R8: value 1k -> 10k
Connections:
- net +3V3: now also R12.1, R14.2, R15.2
- net GND: now also J3.2 (Pin_2), R13.2
- net MOTOR_M: now also J3.1 (Pin_1)
- net MOTOR_P: now also J3.6 (Pin_6)
- net at R10.1: now also J3.3 (Pin_3)
- net at R11.1: now also J3.4 (Pin_4)
- net at FB1.1: now also J3.5 (Pin_5)
- net ADDR: now reaches U1.19 (PA03)
- net ADDR: now also R12.2, R13.1
- net FNC1 renamed STOP_1
- net STOP_1: now also J3.7 (Pin_7), R14.1
- net FNC2 renamed STOP_2
- net STOP_2: now also J3.8 (Pin_8), R15.1
- no-connect marks 2 -> 1
Other:
- note added: "pullup k STOP1/2"
- note added: "zmenit velikost R7, R8"
- moved on the sheet: D2, D3, FB1, R10, R11, R7, R8
