File: t100-raspi/board/t100-raspi.sch (KiCad schematic (older format))
At the start: 8 parts, among them J1 Raspberry_Pi_2_3, J2 12V, J3 USB_B_Micro, J4 UART, J5 T100-OUT, U1 CH330N

Commit message: WIP
Parts:
- removed J5: T100-OUT, Connector_PinSocket_2.54mm:PinSocket_1x12_P2.54mm_Horizontal, symbol t100-raspi-rescue:T100-OUT-device.farm
- added C10, C3, C4, C9: 100u/12V, Capacitor_SMD:CP_Elec_6.3x5.4, symbol Device:CP
- added C5, C6, C7, C8: 100n, Capacitor_SMD:C_0805_2012Metric, symbol Device:C
- added DG1: GREEN, LED_SMD:LED_0805_2012Metric_Pad1.15x1.40mm_HandSolder, symbol Device:LED
- added DR1: RED, LED_SMD:LED_0805_2012Metric_Pad1.15x1.40mm_HandSolder, symbol Device:LED
- added DW1: WHITE, LED_SMD:LED_0805_2012Metric_Pad1.15x1.40mm_HandSolder, symbol Device:LED
- added DY1: YELLOW, LED_SMD:LED_0805_2012Metric_Pad1.15x1.40mm_HandSolder, symbol Device:LED
- added J5: T100-OUT, Connector_PinSocket_2.54mm:PinSocket_1x12_P2.54mm_Horizontal, symbol device.farm:T100-OUT
- added L1, L2: 6.8uH, device.farm:CKCS6028, symbol Device:L
- added R1, R2: 100k, Resistor_SMD:R_0805_2012Metric, symbol Device:R
- added R10: 6.65k 1%, Resistor_SMD:R_0805_2012Metric, symbol Device:R
- added R11, R12, R13, R14: 270R, Resistor_SMD:R_0805_2012Metric, symbol Device:R
- added R3, R4, R5, R6: 1K5, Resistor_SMD:R_0805_2012Metric, symbol Device:R
- added R7: 30.9k 1%, Resistor_SMD:R_0805_2012Metric, symbol Device:R
- added R8: 4.22k 1%, Resistor_SMD:R_0805_2012Metric, symbol Device:R
- added R9: 30k 1%, Resistor_SMD:R_0805_2012Metric, symbol Device:R
- added U2, U3: FR8205, Package_TO_SOT_SMD:SOT-23-6, symbol device.farm:FR8205
- J4: renamed from J2; footprint device.farm:DG142R-2-5.08 -> device.farm:DG301-5.0-02
- renumbered J3 to J1, J4 to J2, J1 to J3
Connections:
- net labels added: I2C_ACT
- wire segments 25 -> 99
Other:
- moved on the sheet: C1, C2, J1, J2, J3, J4, U1

Commit message: WIP
Parts:
- removed DG1: GREEN, LED_SMD:LED_0805_2012Metric_Pad1.15x1.40mm_HandSolder, symbol Device:LED
- removed DR1: RED, LED_SMD:LED_0805_2012Metric_Pad1.15x1.40mm_HandSolder, symbol Device:LED
- removed DW1: WHITE, LED_SMD:LED_0805_2012Metric_Pad1.15x1.40mm_HandSolder, symbol Device:LED
- removed DY1: YELLOW, LED_SMD:LED_0805_2012Metric_Pad1.15x1.40mm_HandSolder, symbol Device:LED
- removed R11, R12, R13, R14: 270R, Resistor_SMD:R_0805_2012Metric, symbol Device:R
Connections:
- net IRQ: now also J3.29 (GCLK1/GPIO5)
- net SCL: now also J3.5 (SCL/GPIO3)
- net SDA: now also J3.3 (SDA/GPIO2)
- net TRG: now also J3.31 (GCLK2/GPIO6)
- no-connect marks 4 -> 26
Other:
- moved on the sheet: R3, R4, R5, R6

Commit message: WIP
Parts:
- R10: value 6.65k 1% -> 4.22k 1%
- R7: value 30.9k 1% -> 30k 1%
- R8: value 4.22k 1% -> 6.65k 1%
- R9: value 30k 1% -> 30.9k 1%
Connections:
- net +3V3: now also C9.1, L1.2, R7.2; no longer C10.1, L2.2, R9.2
- net +5V: now also C10.1, L2.2, R9.2; no longer C9.1, L1.2, R7.2
Changed lines of the file:
@@
 P 7300 1650
 F 0 "R7" H 7200 1650 50  0000 C CNN
-F 1 "30.9k 1%" H 7550 1650 50  0000 C CNN
+F 1 "30k 1%" H 7550 1650 50  0000 C CNN
 F 2 "Resistor_SMD:R_0805_2012Metric" V 7230 1650 50  0001 C CNN
 F 3 "" H 7300 1650 50  0001 C CNN
@@
 P 7300 2050
 F 0 "R8" H 7200 2050 50  0000 C CNN
-F 1 "4.22k 1%" H 7550 2050 50  0000 C CNN
+F 1 "6.65k 1%" H 7550 2050 50  0000 C CNN
 F 2 "Resistor_SMD:R_0805_2012Metric" V 7230 2050 50  0001 C CNN
 F 3 "" H 7300 2050 50  0001 C CNN
@@
 L power:+5V #PWR020
 U 1 1 5CC9CAD4
-P 7850 1450
-F 0 "#PWR020" H 7850 1300 50  0001 C CNN
-F 1 "+5V" H 7850 1590 50  0000 C CNN
-F 2 "" H 7850 1450 50  0001 C CNN
-F 3 "" H 7850 1450 50  0001 C CNN
-	1    7850 1450
+P 7850 3150
+F 0 "#PWR020" H 7850 3000 50  0001 C CNN
+F 1 "+5V" H 7850 3290 50  0000 C CNN
+F 2 "" H 7850 3150 50  0001 C CNN
+F 3 "" H 7850 3150 50  0001 C CNN
+	1    7850 3150
 	0    1    1    0
 $EndComp
@@
 P 7300 3350
 F 0 "R9" H 7200 3350 50  0000 C CNN
-F 1 "30k 1%" H 7550 3350 50  0000 C CNN
+F 1 "30.9k 1%" H 7550 3350 50  0000 C CNN
 F 2 "Resistor_SMD:R_0805_2012Metric" V 7230 3350 50  0001 C CNN
 F 3 "" H 7300 3350 50  0001 C CNN
@@
 P 7300 3750
 F 0 "R10" H 7200 3750 50  0000 C CNN
-F 1 "6.65k 1%" H 7550 3750 50  0000 C CNN
+F 1 "4.22k 1%" H 7550 3750 50  0000 C CNN
 F 2 "Resistor_SMD:R_0805_2012Metric" V 7230 3750 50  0001 C CNN
 F 3 "" H 7300 3750 50  0001 C CNN
@@
 L power:+3V3 #PWR021
 U 1 1 6012C0E5
-P 7850 3150
-F 0 "#PWR021" H 7850 3000 50  0001 C CNN
-F 1 "+3V3" V 7865 3278 50  0000 L CNN
-F 2 "" H 7850 3150 50  0001 C CNN
-F 3 "" H 7850 3150 50  0001 C CNN
-	1    7850 3150
+P 7850 1450
+F 0 "#PWR021" H 7850 1300 50  0001 C CNN
+F 1 "+3V3" V 7865 1578 50  0000 L CNN
+F 2 "" H 7850 1450 50  0001 C CNN
+F 3 "" H 7850 1450 50  0001 C CNN
+	1    7850 1450
 	0    1    1    0
 $EndComp

Commit message: WIP
Parts:
- added C11: 100n, Capacitor_SMD:C_0805_2012Metric, symbol Device:C
- J1: footprint device.farm:conn_usb_B_micro_smd-2 -> Drake:conn_usb_B_micro_smd-2
- J3: footprint device.farm:Raspberry-PI-3-B-vertical -> Drake:Raspberry-PI-3-B-vertical
- J4: footprint device.farm:DG301-5.0-02 -> Drake:DG301-5.0-02
- J5: symbol device.farm:T100-OUT -> Drake:T100-OUT
- L1, L2: footprint device.farm:CKCS6028 -> Drake:CKCS6028
- U2, U3: symbol device.farm:FR8205 -> Drake:FR8205
Connections:
- net +12V: now also J5.8 (12V), J5.9 (12V); no longer J5.10 (12V), J5.11 (12V)
- net +5V: now also J5.7 (5V); no longer J5.8 (5V)
- net GND: now also J5.10 (GND), C11.2; no longer J5.12 (GND), J5.7 (GND), J5.9 (GND)
- net TRG renamed RST
- net RST: now also C11.1
Changed lines of the file:
@@
 F 0 "J3" H 3050 7150 50  0000 C CNN
 F 1 "Raspberry_Pi_2_3" H 3300 7050 50  0000 C CNN
-F 2 "device.farm:Raspberry-PI-3-B-vertical" H 2550 5650 50  0001 C CNN
+F 2 "Drake:Raspberry-PI-3-B-vertical" H 2550 5650 50  0001 C CNN
 F 3 "https://www.raspberrypi.org/documentation/hardware/raspberrypi/schematics/rpi_SCH_3bplus_1p0_reduced.pdf" H 2550 5650 50  0001 C CNN
 	1    2550 5650
@@
 F 0 "J4" H 2642 2975 50  0000 C CNN
 F 1 "12V" H 2642 3066 50  0000 C CNN
-F 2 "device.farm:DG301-5.0-02" H 2750 3300 50  0001 C CNN
+F 2 "Drake:DG301-5.0-02" H 2750 3300 50  0001 C CNN
 F 3 "~" H 2750 3300 50  0001 C CNN
 	1    2750 3300
@@
 F 0 "J1" H 1607 2167 50  0000 C CNN
 F 1 "USB_B_Micro" H 1607 2076 50  0000 C CNN
-F 2 "device.farm:conn_usb_B_micro_smd-2" H 1700 1650 50  0001 C CNN
+F 2 "Drake:conn_usb_B_micro_smd-2" H 1700 1650 50  0001 C CNN
 F 3 "~" H 1700 1650 50  0001 C CNN
 	1    1550 1700
@@
 IRQ
 Text Label 3350 5550 0    50   ~ 0
-TRG
+RST
 Text Label 3600 1500 0    50   ~ 0
 MY_RXD
@@
 F 0 "L1" V 7100 1450 50  0000 C CNN
 F 1 "6.8uH" V 7225 1450 50  0000 C CNN
-F 2 "device.farm:CKCS6028" H 7150 1450 50  0001 C CNN
+F 2 "Drake:CKCS6028" H 7150 1450 50  0001 C CNN
 F 3 "" H 7150 1450 50  0001 C CNN
 	1    7150 1450
@@
 	7300 1500 7300 1450
 $Comp
-L device.farm:FR8205 U2
+L Drake:FR8205 U2
 U 1 1 5CC26308
 P 6400 1750
@@
 F 0 "L2" V 7100 3150 50  0000 C CNN
 F 1 "6.8uH" V 7225 3150 50  0000 C CNN
-F 2 "device.farm:CKCS6028" H 7150 3150 50  0001 C CNN
+F 2 "Drake:CKCS6028" H 7150 3150 50  0001 C CNN
 F 3 "" H 7150 3150 50  0001 C CNN
 	1    7150 3150
@@
 	7300 3200 7300 3150
 $Comp
-L device.farm:FR8205 U3
+L Drake:FR8205 U3
 U 1 1 60129439
 P 6400 3450
@@
 $EndComp
 $Comp
-L device.farm:T100-OUT J5
+L Drake:T100-OUT J5
 U 1 1 601332C1
-P 10250 2200
-F 0 "J5" H 10428 2246 50  0000 L CNN
-F 1 "T100-OUT" H 10428 2155 50  0000 L CNN
-F 2 "Connector_PinSocket_2.54mm:PinSocket_1x12_P2.54mm_Horizontal" H 10250 1300 50  0001 C CNN
-F 3 "" H 10250 2200 50  0001 C CNN
-	1    10250 2200
+P 10150 2100
+F 0 "J5" H 10450 2150 50  0000 L CNN
+F 1 "T100-OUT" H 10450 2050 50  0000 L CNN
+F 2 "Connector_PinSocket_2.54mm:PinSocket_1x12_P2.54mm_Horizontal" H 10150 1200 50  0001 C CNN
+F 3 "" H 10150 2100 50  0001 C CNN
+	1    10150 2100
 	1    0    0    -1
 $EndComp
@@
 	0    -1   -1   0
 $EndComp
-Wire Wire Line
-	10050 2550 10050 2650
-Connection ~ 10050 2650
-Wire Wire Line
-	10050 2650 10050 2750
-Connection ~ 10050 2750
-Wire Wire Line
-	10050 2750 10050 2850
-Connection ~ 10050 2850
-Wire Wire Line
-	10050 2850 10050 3050
 $Comp
 L power:GND #PWR031
 U 1 1 601364DD
-P 10050 3050
-F 0 "#PWR031" H 10050 2800 50  0001 C CNN
-F 1 "GND" H 10050 2900 50  0000 C CNN
-F 2 "" H 10050 3050 50  0001 C CNN
-F 3 "" H 10050 3050 50  0001 C CNN
-	1    10050 3050
+P 10050 2650
+F 0 "#PWR031" H 10050 2400 50  0001 C CNN
+F 1 "GND" H 10050 2500 50  0000 C CNN
+F 2 "" H 10050 2650 50  0001 C CNN
+F 3 "" H 10050 2650 50  0001 C CNN
+	1    10050 2650
 	1    0    0    -1
 $EndComp
@@
 IRQ
 Text Label 10050 2400 2    50   ~ 0
-TRG
+RST
 $Comp
 L Device:R R3
@@
 	5100 6150 5000 6150
 Text Label 5000 6150 2    50   ~ 0
-TRG
+RST
 NoConn ~ 3350 5750
 NoConn ~ 3350 5850
@@
 NoConn ~ 3350 4850
 NoConn ~ 3350 4750
+Wire Wire Line
+	10050 2550 10050 2650
+Connection ~ 10050 2650
+$Comp
+L Device:C C11
+U 1 1 6073999A
+P 5000 6300
+F 0 "C11" H 4700 6250 50  0000 L CNN
+F 1 "100n" H 4650 6350 50  0000 L CNN
+F 2 "Capacitor_SMD:C_0805_2012Metric" H 5038 6150 50  0001 C CNN
+F 3 "" H 5000 6300 50  0001 C CNN
+	1    5000 6300
+	1    0    0    -1
+$EndComp
+$Comp
+L power:GND #PWR022
+U 1 1 6073A10F
+P 5000 6450
+F 0 "#PWR022" H 5000 6200 50  0001 C CNN
+F 1 "GND" H 5000 6300 50  0000 C CNN
+F 2 "" H 5000 6450 50  0001 C CNN
+F 3 "" H 5000 6450 50  0001 C CNN
+	1    5000 6450
+	1    0    0    -1
+$EndComp
 $EndSCHEMATC
