File: t100-raspi/board/t100-raspi.kicad_pcb (KiCad board)
At the start: 2 copper layers, 49.5 x 99.5 mm, 30 parts, among them J1 USB_B_Micro, J2 UART, J3 Raspberry_Pi_2_3, J4 12V, J5 T100-OUT, U1 CH330N, U2 FR8205, U3 FR8205

Commit message: WIP
Parts:
- moved C6 153.6 mm to (95.0, 60.0), turned to 90 degrees
- moved C8 140.3 mm to (99.0, 52.0)
- moved C1 137.2 mm to (42.5, 62.2)
- moved C10 137.2 mm to (54.0, 48.6)
- moved C2 137.2 mm to (37.8, 62.2)
- moved J1 137.2 mm to (54.1, 32.7)
- moved R10 132.0 mm to (99.0, 63.0)
- moved R9 123.6 mm to (103.0, 63.0)
- moved R2 109.9 mm to (103.0, 58.0), turned to 90 degrees
- moved U3 109.8 mm to (99.0, 56.0)
- moved C4 100.1 mm to (90.0, 55.0), turned to 180 degrees
- moved L2 83.6 mm to (108.0, 56.0), turned to 270 degrees
- moved U1 58.2 mm to (148.0, 30.0)
Routing:
- net +12V: track 0.00 -> 47.2 mm
- net +3V3: track 0.00 -> 35.7 mm
- net Net-(C8-Pad2): track 0.00 -> 11.8 mm
- net Net-(R2-Pad1): track 0.00 -> 3.72 mm
- net Net-(C8-Pad1): track 0.00 -> 3.12 mm
- net Net-(R10-Pad2): track 0.00 -> 2.12 mm
Other:
- net class Default: trace_width 0.25 -> 0.4

Commit message: WIP
Parts:
- R10: value 6.65k 1% -> 4.22k 1%
- R7: value 30.9k 1% -> 30k 1%
- R8: value 4.22k 1% -> 6.65k 1%
- R9: value 30k 1% -> 30.9k 1%
- moved J1 128.1 mm to (110.0, 148.0)
- moved U1 114.8 mm to (110.5, 138.5), turned to 90 degrees
- moved C2 108.2 mm to (115.0, 138.0), turned to 270 degrees
- moved C1 106.6 mm to (117.5, 138.0), turned to 270 degrees
- moved J2 103.0 mm to (122.0, 136.5), turned to 180 degrees
- moved C10 57.9 mm to (111.5, 55.5), turned to 90 degrees
- moved R5 53.7 mm to (110.5, 91.2), turned to 270 degrees
- moved R6 47.5 mm to (111.5, 80.9), turned to 90 degrees
- moved R3 37.6 mm to (109.4, 77.5)
- moved J4 37.3 mm to (92.5, 53.5), turned to 180 degrees
- moved R4 36.5 mm to (111.5, 74.0), turned to 270 degrees
- moved R10 10.8 mm to (108.0, 69.0)
- moved C4 9.01 mm to (95.0, 62.5), turned to 0 degrees
- moved R9 7.02 mm to (110.0, 62.5)
- moved C6 6.08 mm to (89.0, 59.0), turned to 180 degrees
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Connections:
- C10 pad 1: +3V3 -> +5V
- C9 pad 1: +5V -> +3V3
- L1 pad 2: +5V -> +3V3
- L2 pad 2: +3V3 -> +5V
- R7 pad 2: +5V -> +3V3
- R9 pad 2: +3V3 -> +5V
Routing:
- net /MY_TXD: track 0.00 -> 80.5 mm, vias 0 -> 2
- net /MY_RXD: track 0.00 -> 76.3 mm
- net +12V: track 47.2 -> 119.2 mm, vias 0 -> 3
- net GND: track 0.00 -> 66.2 mm, vias 0 -> 16
- net +5V: track 0.00 -> 55.5 mm
- net +3V3: track 35.7 -> 79.3 mm
- net /TRG: track 0.00 -> 41.6 mm, vias 0 -> 1
- net /IRQ: track 0.00 -> 41.5 mm, vias 0 -> 2
- net Net-(R10-Pad2): track 2.12 -> 34.9 mm, vias 0 -> 3
- net Net-(C1-Pad1): track 0.00 -> 29.7 mm, vias 0 -> 2
- net /SDA: track 0.00 -> 24.8 mm
- net /SCL: track 0.00 -> 21.9 mm
- net Net-(J1-Pad2): track 0.00 -> 11.0 mm
- net Net-(C7-Pad2): track 0.00 -> 8.88 mm
- net Net-(C2-Pad1): track 0.00 -> 8.27 mm
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- added copper zone on B.Cu, net GND

Commit message: WIP
Routing:
- net GND: track 66.2 -> 83.2 mm, vias 16 -> 27
- net +12V: track 119.2 -> 124.5 mm, vias 3 -> 6
Other:
- outline, holes or cut-outs redrawn
- board text added: "+12V"
- board text added: "G"
- board text added: "GND"
- board text added: "RX"
- board text added: "T100-RASPI v1"
- board text added: "TX"
- board text added: "UART"

Commit message: WIP
Parts:
- J1: footprint device.farm:conn_usb_B_micro_smd-2 -> Drake:conn_usb_B_micro_smd-2
- J3: footprint device.farm:Raspberry-PI-3-B-vertical -> Drake:Raspberry-PI-3-B-vertical
- J4: footprint device.farm:DG301-5.0-02 -> Drake:DG301-5.0-02
- L1, L2: footprint device.farm:CKCS6028 -> Drake:CKCS6028
Changed lines of the file:
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@@
     (add_net "Net-(U1-Pad4)")
   )
-  (module device.farm:Raspberry-PI-3-B-vertical (layer F.Cu)
+  (module Drake:Raspberry-PI-3-B-vertical (layer F.Cu)
     (at 104 69 90)
     (fp_text reference J3 (at 5.08 -7.62 90) (layer F.SilkS)
@@
     )
   )
-  (module device.farm:CKCS6028 (layer F.Cu)
+  (module Drake:CKCS6028 (layer F.Cu)
     (at 104 56 270)
     (descr "Inductor, Taiyo Yuden, NR series, Taiyo-Yuden_NR-60xx, 6.0mmx6.0mm")
@@
     )
   )
-  (module device.farm:CKCS6028 (layer F.Cu)
+  (module Drake:CKCS6028 (layer F.Cu)
     (at 115 115)
     (descr "Inductor, Taiyo Yuden, NR series, Taiyo-Yuden_NR-60xx, 6.0mmx6.0mm")
@@
     )
   )
-  (module device.farm:DG301-5.0-02 (layer F.Cu)
+  (module Drake:DG301-5.0-02 (layer F.Cu)
     (at 92.5 53.5 180)
     (fp_text reference J4 (at 8.5 -3) (layer F.SilkS)
@@
     )
   )
-  (module device.farm:conn_usb_B_micro_smd-2 (layer F.Cu)
+  (module Drake:conn_usb_B_micro_smd-2 (layer F.Cu)
     (at 110 148)
     (descr "USB B micro SMD connector with retention pins")

Commit message: WIP
Parts:
- added C11: 100n, Capacitor_SMD:C_0805_2012Metric, F.Cu at (108.0, 116.6)
- J5: footprint Connector_PinSocket_2.54mm:PinSocket_1x12_P2.54mm_Horizontal -> Connector_PinSocket_2.54mm:PinSocket_1x10_P2.54mm_Horizontal
- moved R4 2.10 mm to (109.4, 73.6), turned to 0 degrees
- moved R7 2.02 mm to (121.0, 108.1)
- moved R8 2.02 mm to (121.0, 104.1)
Connections:
- net /TRG renamed /RST
- J1 pad 4: Net-(J1-Pad4) -> unconnected-(J1-Pad4)
- J3 pad 1: Net-(J3-Pad1) -> unconnected-(J3-Pad1)
- J3 pad 11: Net-(J3-Pad11) -> unconnected-(J3-Pad11)
- J3 pad 12: Net-(J3-Pad12) -> unconnected-(J3-Pad12)
- J3 pad 13: Net-(J3-Pad13) -> unconnected-(J3-Pad13)
- J3 pad 15: Net-(J3-Pad15) -> unconnected-(J3-Pad15)
- J3 pad 16: Net-(J3-Pad16) -> unconnected-(J3-Pad16)
- J3 pad 17: Net-(J3-Pad17) -> unconnected-(J3-Pad17)
- J3 pad 18: Net-(J3-Pad18) -> unconnected-(J3-Pad18)
- J3 pad 19: Net-(J3-Pad19) -> unconnected-(J3-Pad19)
- J3 pad 21: Net-(J3-Pad21) -> unconnected-(J3-Pad21)
- J3 pad 22: Net-(J3-Pad22) -> unconnected-(J3-Pad22)
- J3 pad 23: Net-(J3-Pad23) -> unconnected-(J3-Pad23)
- J3 pad 24: Net-(J3-Pad24) -> unconnected-(J3-Pad24)
- J3 pad 26: Net-(J3-Pad26) -> unconnected-(J3-Pad26)
- J3 pad 27: Net-(J3-Pad27) -> unconnected-(J3-Pad27)
- J3 pad 28: Net-(J3-Pad28) -> unconnected-(J3-Pad28)
- J3 pad 32: Net-(J3-Pad32) -> unconnected-(J3-Pad32)
- J3 pad 33: Net-(J3-Pad33) -> unconnected-(J3-Pad33)
- J3 pad 35: Net-(J3-Pad35) -> unconnected-(J3-Pad35)
- J3 pad 36: Net-(J3-Pad36) -> unconnected-(J3-Pad36)
- J3 pad 37: Net-(J3-Pad37) -> unconnected-(J3-Pad37)
- J3 pad 38: Net-(J3-Pad38) -> unconnected-(J3-Pad38)
- J3 pad 40: Net-(J3-Pad40) -> unconnected-(J3-Pad40)
- J3 pad 7: Net-(J3-Pad7) -> unconnected-(J3-Pad7)
- J5 pad 10: +12V -> GND
- J5 pad 7: GND -> +5V
- J5 pad 8: +5V -> +12V
- J5 pad 9: GND -> +12V
- U1 pad 4: Net-(U1-Pad4) -> unconnected-(U1-Pad4)
Routing:
- net Net-(R2-Pad1): track 9.86 -> 25.2 mm, vias 0 -> 2
- net +12V: track 124.5 -> 137.4 mm
- net /RST: track 41.6 -> 51.8 mm
- net +5V: track 55.5 -> 61.7 mm
- net Net-(R7-Pad1): track 5.07 -> 10.7 mm, vias 0 -> 2
- net GND: track 83.2 -> 88.0 mm
- net +3V3: track 79.3 -> 83.2 mm
- net /SDA: track 24.8 -> 22.0 mm
Other:
- net class Default removed
- board text added: "T100-RASPI v1.1"
- board text removed: "T100-RASPI v1"
