File: t100-usb/board/t100-usb.sch (KiCad schematic (older format))
At the start: 37 parts, among them J1 Conn_01x02_Female, J2 USB_B_Micro, J3 T100-OUT, U1 FR8205, U2 FR8205, U3 MCP2221A

Commit message: WIP
Parts:
- removed C7: 220n, Capacitor_SMD:C_0805_2012Metric_Pad1.15x1.40mm_HandSolder, symbol Device:C
- removed U3: MCP2221A, Package_SO:SOIC-14_3.9x8.7mm_P1.27mm, symbol device.farm:MCP2221A
- added U3: ATSAMD11C14A-SS, Package_SO:SOIC-14_3.9x8.7mm_P1.27mm, symbol MCU_Microchip_SAMD:ATSAMD11C14A-SS
- added X1: SWD, Drake:SWD, symbol Drake:SWD
- C6: value 47M -> 100n; footprint Capacitor_SMD:C_0805_2012Metric_Pad1.15x1.40mm_HandSolder -> Capacitor_SMD:C_0805_2012Metric
- J1: footprint device.farm:DG301-5.0-02 -> Drake:DG301-5.0-02
- J2: footprint device.farm:conn_usb_B_micro_smd-2 -> Drake:conn_usb_B_micro_smd-2
- J3: symbol device.farm:T100-OUT -> Drake:T100-OUT
- L1, L3: footprint device.farm:CKCS6028 -> Drake:CKCS6028
- U1, U2: symbol device.farm:FR8205 -> Drake:FR8205
Connections:
- net +12V: no longer J3.10 (12V), J3.11 (12V)
- net +3V3: now also C8.2, U3.12 (VDD); no longer DY1.2 (A), J3.6 (3V3)
- net +5V: no longer J3.8 (5V)
- net GND: now also C6.1, DY1.1 (K), U3.11 (GND), X1.2 (GND); no longer C6.2, J3.1 (GND), J3.12 (GND), J3.7 (GND), J3.9 (GND)
- net I2C_ACT: now also U3.13 (PA02)
- net IRQ: now also U3.1 (PA05); no longer J3.4 (IRQ)
- net SCL: now also U3.5 (PA15); no longer J3.2 (SCL)
- net SDA: now also U3.4 (PA14); no longer J3.3 (SDA)
- net TRG: now also U3.14 (PA04); no longer J3.5 (TRG)
- net USB_DM: now reaches J2.2 (D-)
- net USB_DM: now also U3.9 (PA24)
- net USB_DP: now reaches J2.3 (D+)
- net USB_DP: now also U3.10 (PA25)
- net at R4.2: now also DY1.2 (A); no longer DY1.1 (K)
- new net: C6.2, U3.6 (PA28/~RST)
- new net SWCLK: U3.7 (PA30/SWCLK), X1.3 (SWCLK)
- new net SWDIO: U3.8 (PA31/SWDIO), X1.1 (SWDIO)
- now unconnected: J2.1 (VBUS)
- no-connect marks 5 -> 4
Other:
- moved on the sheet: C8, DY1, J2

Commit message: WIP
Parts:
- removed DG1: GREEN, LED_SMD:LED_0805_2012Metric_Pad1.15x1.40mm_HandSolder, symbol Device:LED
- removed R14: 270R, Resistor_SMD:R_0805_2012Metric, symbol Device:R
- added C7: 100n, Capacitor_SMD:C_0805_2012Metric, symbol Device:C
- C1, C19, C4, C5: symbol Device:CP -> Device:C_Polarized
- DG1: renamed from DY1; value YELLOW -> GREEN
- J3: footprint Connector_PinSocket_2.54mm:PinSocket_1x12_P2.54mm_Horizontal -> Connector_PinSocket_2.54mm:PinSocket_1x10_P2.54mm_Horizontal
- R12: value 270R -> 1k5
Connections:
- net TRG is gone; now on net RST: R11.1, U3.14 (PA04)
- net +12V: now also J3.8 (12V), J3.9 (12V)
- net +3V3: now also J3.6 (3V3)
- net +5V: now also J3.7 (5V)
- net GND: now also J3.1 (GND), J3.10 (GND), C7.1
- net IRQ: now also J3.4 (IRQ)
- net SCL: now also J3.2 (SCL)
- net SDA: now also J3.3 (SDA)
- net RST: now reaches J3.5 (RST)
- net RST: now also C7.2
Other:
- moved on the sheet: DG1, DR1, DW1, J3, R12, R13, R4
Changed lines of the file:
@@
 $EndComp
 $Comp
-L Device:CP C4
+L Device:C_Polarized C4
 U 1 1 5CC2AB6A
 P 4400 1850
@@
 	5350 2200 5350 2300
 $Comp
-L Device:CP C19
+L Device:C_Polarized C19
 U 1 1 5CC90415
 P 6650 1850
@@
 $EndComp
 $Comp
-L Device:CP C1
+L Device:C_Polarized C1
 U 1 1 601293F2
 P 4400 3750
@@
 	5350 4100 5350 4200
 $Comp
-L Device:CP C5
+L Device:C_Polarized C5
 U 1 1 60129449
 P 6650 3750
@@
 L Drake:T100-OUT J3
 U 1 1 601332C1
-P 8850 2550
-F 0 "J3" H 9028 2596 50  0000 L CNN
-F 1 "T100-OUT" H 9028 2505 50  0000 L CNN
-F 2 "Connector_PinSocket_2.54mm:PinSocket_1x12_P2.54mm_Horizontal" H 8850 1650 50  0001 C CNN
-F 3 "" H 8850 2550 50  0001 C CNN
-	1    8850 2550
+P 8750 2450
+F 0 "J3" H 9050 2500 50  0000 L CNN
+F 1 "T100-OUT" H 9050 2400 50  0000 L CNN
+F 2 "Connector_PinSocket_2.54mm:PinSocket_1x10_P2.54mm_Horizontal" H 8750 1550 50  0001 C CNN
+F 3 "" H 8750 2450 50  0001 C CNN
+	1    8750 2450
 	1    0    0    -1
 $EndComp
@@
 	0    -1   -1   0
 $EndComp
-Wire Wire Line
-	8650 2900 8650 3000
-Connection ~ 8650 3000
-Wire Wire Line
-	8650 3000 8650 3100
-Connection ~ 8650 3100
-Wire Wire Line
-	8650 3100 8650 3200
-Connection ~ 8650 3200
-Wire Wire Line
-	8650 3200 8650 3400
 $Comp
 L power:GND #PWR016
 U 1 1 601364DD
-P 8650 3400
-F 0 "#PWR016" H 8650 3150 50  0001 C CNN
-F 1 "GND" H 8650 3250 50  0000 C CNN
-F 2 "" H 8650 3400 50  0001 C CNN
-F 3 "" H 8650 3400 50  0001 C CNN
-	1    8650 3400
+P 8650 3000
+F 0 "#PWR016" H 8650 2750 50  0001 C CNN
+F 1 "GND" H 8650 2850 50  0000 C CNN
+F 2 "" H 8650 3000 50  0001 C CNN
+F 3 "" H 8650 3000 50  0001 C CNN
+	1    8650 3000
 	1    0    0    -1
 $EndComp
@@
 Text Label 8650 2650 2    50   ~ 0
 IRQ
-Text Label 8650 2750 2    50   ~ 0
-TRG
 $Comp
 L Connector:USB_B_Micro J2
@@
 IRQ
 Text Label 5150 5650 0    50   ~ 0
-TRG
+RST
 NoConn ~ 2050 4950
 $Comp
 L Device:R R4
 U 1 1 60166CD6
-P 8850 4350
-F 0 "R4" V 9050 4350 50  0000 C CNN
-F 1 "270R" V 8950 4350 50  0000 C CNN
-F 2 "Resistor_SMD:R_0805_2012Metric" V 8780 4350 50  0001 C CNN
-F 3 "" H 8850 4350 50  0001 C CNN
-	1    8850 4350
-	0    -1   -1   0
-$EndComp
-Wire Wire Line
-	8550 4350 8700 4350
-Text Label 8550 4350 2    50   ~ 0
+P 8850 4400
+F 0 "R4" V 9050 4400 50  0000 C CNN
+F 1 "270R" V 8950 4400 50  0000 C CNN
+F 2 "Resistor_SMD:R_0805_2012Metric" V 8780 4400 50  0001 C CNN
+F 3 "" H 8850 4400 50  0001 C CNN
+	1    8850 4400
+	0    -1   -1   0
+$EndComp
+Wire Wire Line
+	8550 4400 8700 4400
+Text Label 8550 4400 2    50   ~ 0
 I2C_ACT
 Text Label 5150 5550 0    50   ~ 0
@@
 L Device:R R13
 U 1 1 60187F28
-P 8850 4800
-F 0 "R13" V 9050 4800 50  0000 C CNN
-F 1 "270R" V 8950 4800 50  0000 C CNN
-F 2 "Resistor_SMD:R_0805_2012Metric" V 8780 4800 50  0001 C CNN
-F 3 "" H 8850 4800 50  0001 C CNN
-	1    8850 4800
+P 8850 5000
+F 0 "R13" V 9050 5000 50  0000 C CNN
+F 1 "270R" V 8950 5000 50  0000 C CNN
+F 2 "Resistor_SMD:R_0805_2012Metric" V 8780 5000 50  0001 C CNN
+F 3 "" H 8850 5000 50  0001 C CNN
+	1    8850 5000
 	0    -1   -1   0
 $EndComp
@@
 L Device:LED DR1
 U 1 1 60187F32
-P 9150 4800
-F 0 "DR1" H 9143 4545 50  0000 C CNN
-F 1 "RED" H 9143 4636 50  0000 C CNN
-F 2 "LED_SMD:LED_0805_2012Metric_Pad1.15x1.40mm_HandSolder" H 9150 4800 50  0001 C CNN
-F 3 "~" H 9150 4800 50  0001 C CNN
-	1    9150 4800
+P 9150 5000
+F 0 "DR1" H 9143 4745 50  0000 C CNN
+F 1 "RED" H 9143 4836 50  0000 C CNN
+F 2 "LED_SMD:LED_0805_2012Metric_Pad1.15x1.40mm_HandSolder" H 9150 5000 50  0001 C CNN
+F 3 "~" H 9150 5000 50  0001 C CNN
+	1    9150 5000
 	1    0    0    1
 $EndComp
-Text Label 8550 4800 2    50   ~ 0
+Text Label 8550 5000 2    50   ~ 0
 IRQ
 $Comp
 L power:+3V3 #PWR024
 U 1 1 60187F3F
-P 9300 4800
-F 0 "#PWR024" H 9300 4650 50  0001 C CNN
-F 1 "+3V3" V 9315 4928 50  0000 L CNN
-F 2 "" H 9300 4800 50  0001 C CNN
-F 3 "" H 9300 4800 50  0001 C CNN
-	1    9300 4800
-	0    1    1    0
-$EndComp
-$Comp
-L Device:R R14
-U 1 1 601C6018
-P 8850 5250
-F 0 "R14" V 9050 5250 50  0000 C CNN
-F 1 "270R" V 8950 5250 50  0000 C CNN
-F 2 "Resistor_SMD:R_0805_2012Metric" V 8780 5250 50  0001 C CNN
-F 3 "" H 8850 5250 50  0001 C CNN
-	1    8850 5250
-	0    -1   -1   0
-$EndComp
-$Comp
-L Device:LED DG1
-U 1 1 601C6022
-P 9150 5250
-F 0 "DG1" H 9143 4995 50  0000 C CNN
-F 1 "GREEN" H 9143 5086 50  0000 C CNN
-F 2 "LED_SMD:LED_0805_2012Metric_Pad1.15x1.40mm_HandSolder" H 9150 5250 50  0001 C CNN
-F 3 "~" H 9150 5250 50  0001 C CNN
-	1    9150 5250
-	1    0    0    1
-$EndComp
-Text Label 8550 5250 2    50   ~ 0
-TRG
-$Comp
-L power:+3V3 #PWR026
-U 1 1 601C602F
-P 9300 5250
-F 0 "#PWR026" H 9300 5100 50  0001 C CNN
-F 1 "+3V3" V 9315 5378 50  0000 L CNN
-F 2 "" H 9300 5250 50  0001 C CNN
-F 3 "" H 9300 5250 50  0001 C CNN
-	1    9300 5250
+P 9300 5000
+F 0 "#PWR024" H 9300 4850 50  0001 C CNN
+F 1 "+3V3" V 9315 5128 50  0000 L CNN
+F 2 "" H 9300 5000 50  0001 C CNN
+F 3 "" H 9300 5000 50  0001 C CNN
+	1    9300 5000
 	0    1    1    0
 $EndComp
@@
 SDA
 Wire Wire Line
-	8550 5250 8700 5250
-Wire Wire Line
-	8550 4800 8700 4800
+	8550 5000 8700 5000
 $Comp
 L Device:R R10
@@
 	6700 6050 6600 6050
 Text Label 6600 6050 2    50   ~ 0
-TRG
+RST
 $Comp
 L power:+3V3 #PWR022
 U 1 1 602082A9
-P 8750 5800
-F 0 "#PWR022" H 8750 5650 50  0001 C CNN
-F 1 "+3V3" V 8765 5928 50  0000 L CNN
-F 2 "" H 8750 5800 50  0001 C CNN
-F 3 "" H 8750 5800 50  0001 C CNN
-	1    8750 5800
+P 8700 5600
+F 0 "#PWR022" H 8700 5450 50  0001 C CNN
+F 1 "+3V3" V 8715 5728 50  0000 L CNN
+F 2 "" H 8700 5600 50  0001 C CNN
+F 3 "" H 8700 5600 50  0001 C CNN
+	1    8700 5600
 	0    -1   -1   0
 $EndComp
@@
 L Device:R R12
 U 1 1 6020898A
-P 9200 5800
-F 0 "R12" V 9400 5800 50  0000 C CNN
-F 1 "270R" V 9300 5800 50  0000 C CNN
-F 2 "Resistor_SMD:R_0805_2012Metric" V 9130 5800 50  0001 C CNN
-F 3 "" H 9200 5800 50  0001 C CNN
-	1    9200 5800
+P 9150 5600
+F 0 "R12" V 9350 5600 50  0000 C CNN
+F 1 "1k5" V 9250 5600 50  0000 C CNN
+F 2 "Resistor_SMD:R_0805_2012Metric" V 9080 5600 50  0001 C CNN
+F 3 "" H 9150 5600 50  0001 C CNN
+	1    9150 5600
 	0    -1   -1   0
 $EndComp
@@
 L Device:LED DW1
 U 1 1 60209071
-P 8900 5800
-F 0 "DW1" H 8893 5545 50  0000 C CNN
-F 1 "WHITE" H 8893 5636 50  0000 C CNN
-F 2 "LED_SMD:LED_0805_2012Metric_Pad1.15x1.40mm_HandSolder" H 8900 5800 50  0001 C CNN
-F 3 "~" H 8900 5800 50  0001 C CNN
-	1    8900 5800
+P 8850 5600
+F 0 "DW1" H 8843 5345 50  0000 C CNN
+F 1 "WHITE" H 8843 5436 50  0000 C CNN
+F 2 "LED_SMD:LED_0805_2012Metric_Pad1.15x1.40mm_HandSolder" H 8850 5600 50  0001 C CNN
+F 3 "~" H 8850 5600 50  0001 C CNN
+	1    8850 5600
 	-1   0    0    1
 $EndComp
@@
 L power:GND #PWR027
 U 1 1 60213956
-P 9350 5800
-F 0 "#PWR027" H 9350 5550 50  0001 C CNN
-F 1 "GND" V 9355 5672 50  0000 R CNN
-F 2 "" H 9350 5800 50  0001 C CNN
-F 3 "" H 9350 5800 50  0001 C CNN
-	1    9350 5800
+P 9300 5600
+F 0 "#PWR027" H 9300 5350 50  0001 C CNN
+F 1 "GND" V 9305 5472 50  0000 R CNN
+F 2 "" H 9300 5600 50  0001 C CNN
+F 3 "" H 9300 5600 50  0001 C CNN
+	1    9300 5600
 	0    -1   -1   0
 $EndComp
@@
 NoConn ~ 2050 4550
 $Comp
-L Device:LED DY1
+L Device:LED DG1
 U 1 1 60167849
-P 9150 4350
-F 0 "DY1" H 9143 4095 50  0000 C CNN
-F 1 "YELLOW" H 9143 4186 50  0000 C CNN
-F 2 "LED_SMD:LED_0805_2012Metric_Pad1.15x1.40mm_HandSolder" H 9150 4350 50  0001 C CNN
-F 3 "~" H 9150 4350 50  0001 C CNN
-	1    9150 4350
-	-1   0    0    1
-$EndComp
-$Comp
-L power:GND #PWR?
+P 9150 4400
+F 0 "DG1" H 9143 4145 50  0000 C CNN
+F 1 "GREEN" H 9143 4236 50  0000 C CNN
+F 2 "LED_SMD:LED_0805_2012Metric_Pad1.15x1.40mm_HandSolder" H 9150 4400 50  0001 C CNN
+F 3 "~" H 9150 4400 50  0001 C CNN
+	1    9150 4400
+	-1   0    0    1
+$EndComp
+$Comp
+L power:GND #PWR0105
 U 1 1 604228F3
-P 9300 4350
-F 0 "#PWR?" H 9300 4100 50  0001 C CNN
-F 1 "GND" V 9305 4222 50  0000 R CNN
-F 2 "" H 9300 4350 50  0001 C CNN
-F 3 "" H 9300 4350 50  0001 C CNN
-	1    9300 4350
-	0    -1   -1   0
+P 9300 4400
+F 0 "#PWR0105" H 9300 4150 50  0001 C CNN
+F 1 "GND" V 9305 4272 50  0000 R CNN
+F 2 "" H 9300 4400 50  0001 C CNN
+F 3 "" H 9300 4400 50  0001 C CNN
+	1    9300 4400
+	0    -1   -1   0
+$EndComp
+Wire Wire Line
+	8650 2900 8650 3000
+Connection ~ 8650 3000
+Text Label 8650 2750 2    50   ~ 0
+RST
+$Comp
+L Device:C C7
+U 1 1 60708A54
+P 6600 6200
+F 0 "C7" H 6800 6150 50  0000 L CNN
+F 1 "100n" H 6750 6250 50  0000 L CNN
+F 2 "Capacitor_SMD:C_0805_2012Metric" H 6638 6050 50  0001 C CNN
+F 3 "" H 6600 6200 50  0001 C CNN
+	1    6600 6200
+	-1   0    0    1
+$EndComp
+$Comp
+L power:GND #PWR0106
+U 1 1 6070915A
+P 6600 6350
+F 0 "#PWR0106" H 6600 6100 50  0001 C CNN
+F 1 "GND" H 6605 6177 50  0000 C CNN
+F 2 "" H 6600 6350 50  0001 C CNN
+F 3 "" H 6600 6350 50  0001 C CNN
+	1    6600 6350
+	1    0    0    -1
 $EndComp
 $EndSCHEMATC
