File: t100-usb/board/t100-usb.kicad_sch (KiCad schematic)
At the start: 36 parts, among them J1 Conn_01x02_Female, J2 USB_B_Micro, J3 T100-OUT, U1 FR8205, U2 FR8205, U3 ATSAMD11C14A-SS, X1 SWD

Commit message: WIP
Parts:
- removed C1, C19, C4, C5: 100u/12V, Capacitor_SMD:CP_Elec_6.3x5.4, symbol Device:C_Polarized
- removed C11, C18, C2, C3: 100n, Capacitor_SMD:C_0805_2012Metric, symbol Device:C
- removed DW1: WHITE, LED_SMD:LED_0805_2012Metric_Pad1.15x1.40mm_HandSolder, symbol Device:LED
- removed J1: Conn_01x02_Female, Drake:DG235-3.81-02P, symbol Connector:Conn_01x02_Female
- removed L1, L3: 6.8uH, Drake:CKCS6028, symbol Device:L
- removed R1, R5: 100k, Resistor_SMD:R_0805_2012Metric, symbol Device:R
- removed R12: 1k5, Resistor_SMD:R_0805_2012Metric, symbol Device:R
- removed R2: 30k 1%, Resistor_SMD:R_0805_2012Metric, symbol Device:R
- removed R3: 6.65k 1%, Resistor_SMD:R_0805_2012Metric, symbol Device:R
- removed R6: 30.9k 1%, Resistor_SMD:R_0805_2012Metric, symbol Device:R
- removed R7: 4.22k 1%, Resistor_SMD:R_0805_2012Metric, symbol Device:R
- removed U1, U2: FR8205, Package_TO_SOT_SMD:SOT-23-6, symbol Drake:FR8205
- added J2: T100-IN, Connector_PinHeader_2.54mm:PinHeader_1x10_P2.54mm_Horizontal, symbol Drake:T100-IN
- renumbered C8 to C1, C6 to C2, C7 to C3, DG1 to D1, DR1 to D2, J2 to J1, R8 to R1, R9 to R2, R10 to R3, R11 to R4, R4 to R5, R13 to R6, U3 to U1
Connections:
- net +12V: now also J2.8 (12V), J2.9 (12V)
- net +3V3: now also J2.6 (3V3)
- net +5V: now also J2.7 (5V)
- net GND: now also J2.1 (GND), J2.10 (GND)
- net IRQ: now also J2.4 (IRQ)
- net RST: now also J2.5 (RST)
- net SCL: now also J2.2 (SCL)
- net SDA: now also J2.3 (SDA)
Other:
- moved on the sheet: J1, X1
