File: t100-usb/board/t100-usb.kicad_pcb (KiCad board)
At the start: 2 copper layers, 34.5 x 99.5 mm, 37 parts, among them J1 Conn_01x02_Female, J2 USB_B_Micro, J3 T100-OUT, U1 FR8205, U2 FR8205, U3 MCP2221A

Commit message: WIP
Other:
- board text added: "+12V"
- board text added: "T100-USB v1"
- board text added: "act"
- board text added: "irq"
- board text added: "pwr"
- board text added: "trg"
Changed lines of the file:
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@@
   (general
     (thickness 1.6)
-    (drawings 30)
+    (drawings 46)
     (tracks 295)
     (zones 0)
@@
     (solder_mask_min_width 0.25)
     (aux_axis_origin 0 0)
-    (grid_origin 107.315 90.17)
     (visible_elements FFFFFF7F)
     (pcbplotparams
@@
     (tags capacitor)
     (attr smd)
-    (fp_text reference C8 (at 0 -1.65) (layer F.SilkS)
+    (fp_text reference C8 (at -2.815 -0.17) (layer F.SilkS)
       (effects (font (size 1 1) (thickness 0.15)))
     )
@@
     (tags SOT-23-6)
     (attr smd)
-    (fp_text reference U2 (at 0 -2.9) (layer F.SilkS)
+    (fp_text reference U2 (at 2.815 -2.33) (layer F.SilkS)
       (effects (font (size 1 1) (thickness 0.15)))
     )
@@
     (tags SOT-23-6)
     (attr smd)
-    (fp_text reference U1 (at 0 -2.9) (layer F.SilkS)
+    (fp_text reference U1 (at 2.815 -2.33) (layer F.SilkS)
       (effects (font (size 1 1) (thickness 0.15)))
     )
@@
     (tags resistor)
     (attr smd)
-    (fp_text reference R12 (at 0 -1.65 90) (layer F.SilkS)
+    (fp_text reference R12 (at 0 1.685 90) (layer F.SilkS)
       (effects (font (size 1 1) (thickness 0.15)))
     )
@@
     (tags resistor)
     (attr smd)
-    (fp_text reference R7 (at 0 -1.65) (layer F.SilkS)
+    (fp_text reference R7 (at -3.185 0.17) (layer F.SilkS)
       (effects (font (size 1 1) (thickness 0.15)))
     )
@@
     (tags resistor)
     (attr smd)
-    (fp_text reference R6 (at 0 -1.65) (layer F.SilkS)
+    (fp_text reference R6 (at 0 1.67) (layer F.SilkS)
       (effects (font (size 1 1) (thickness 0.15)))
     )
@@
     (tags resistor)
     (attr smd)
-    (fp_text reference R3 (at 0 -1.65) (layer F.SilkS)
+    (fp_text reference R3 (at -3.185 0.17) (layer F.SilkS)
       (effects (font (size 1 1) (thickness 0.15)))
     )
@@
     (tags resistor)
     (attr smd)
-    (fp_text reference R2 (at 0 -1.65) (layer F.SilkS)
+    (fp_text reference R2 (at 0 1.67) (layer F.SilkS)
       (effects (font (size 1 1) (thickness 0.15)))
     )
@@
     (tags "capacitor electrolytic")
     (attr smd)
-    (fp_text reference C19 (at 0 -4.35) (layer F.SilkS)
+    (fp_text reference C19 (at 3.185 4.33) (layer F.SilkS)
       (effects (font (size 1 1) (thickness 0.15)))
     )
@@
     (tags "capacitor handsolder")
     (attr smd)
-    (fp_text reference C6 (at 0 -1.65) (layer F.SilkS)
+    (fp_text reference C6 (at 2.815 0.17) (layer F.SilkS)
       (effects (font (size 1 1) (thickness 0.15)))
     )
@@
     (tags "capacitor electrolytic")
     (attr smd)
-    (fp_text reference C5 (at 0 -4.35) (layer F.SilkS)
+    (fp_text reference C5 (at 3.685 4.33) (layer F.SilkS)
       (effects (font (size 1 1) (thickness 0.15)))
     )
@@
     (tags "capacitor electrolytic")
     (attr smd)
-    (fp_text reference C4 (at 0 -4.35) (layer F.SilkS)
+    (fp_text reference C4 (at 3.815 -4.33) (layer F.SilkS)
       (effects (font (size 1 1) (thickness 0.15)))
     )
@@
     (tags "capacitor electrolytic")
     (attr smd)
-    (fp_text reference C1 (at 0 -4.35) (layer F.SilkS)
+    (fp_text reference C1 (at 3.815 -4.33) (layer F.SilkS)
       (effects (font (size 1 1) (thickness 0.15)))
     )
@@
     )
   )
-  (gr_text GND (at 105.41 90.17) (layer F.SilkS)
+  (dimension 17.5 (width 0.15) (layer Dwgs.User)
+    (gr_text "17,500 mm" (at 91.25 46.7) (layer Dwgs.User)
+      (effects (font (size 1 1) (thickness 0.15)))
+    )
+    (feature1 (pts (xy 100 50) (xy 100 47.413579)))
+    (feature2 (pts (xy 82.5 50) (xy 82.5 47.413579)))
+    (crossbar (pts (xy 82.5 48) (xy 100 48)))
+    (arrow1a (pts (xy 100 48) (xy 98.873496 48.586421)))
+    (arrow1b (pts (xy 100 48) (xy 98.873496 47.413579)))
+    (arrow2a (pts (xy 82.5 48) (xy 83.626504 48.586421)))
+    (arrow2b (pts (xy 82.5 48) (xy 83.626504 47.413579)))
+  )
+  (dimension 35 (width 0.15) (layer Dwgs.User)
+    (gr_text "35,000 mm" (at 100 43.2) (layer Dwgs.User)
+      (effects (font (size 1 1) (thickness 0.15)))
+    )
+    (feature1 (pts (xy 117.5 50) (xy 117.5 43.913579)))
+    (feature2 (pts (xy 82.5 50) (xy 82.5 43.913579)))
+    (crossbar (pts (xy 82.5 44.5) (xy 117.5 44.5)))
+    (arrow1a (pts (xy 117.5 44.5) (xy 116.373496 45.086421)))
+    (arrow1b (pts (xy 117.5 44.5) (xy 116.373496 43.913579)))
+    (arrow2a (pts (xy 82.5 44.5) (xy 83.626504 45.086421)))
+    (arrow2b (pts (xy 82.5 44.5) (xy 83.626504 43.913579)))
+  )
+  (gr_text "T100-USB v1" (at 100 55) (layer F.SilkS)
+    (effects (font (size 1.5 1.5) (thickness 0.3)))
+  )
+  (gr_text trg (at 98.815 60.17 45) (layer F.SilkS)
+    (effects (font (size 1.2 1.2) (thickness 0.2)) (justify left))
+  )
+  (gr_text irq (at 95.315 60.17 45) (layer F.SilkS)
+    (effects (font (size 1.2 1.2) (thickness 0.2)) (justify left))
+  )
+  (gr_text act (at 91.815 60 45) (layer F.SilkS)
+    (effects (font (size 1.2 1.2) (thickness 0.2)) (justify left))
+  )
+  (gr_text pwr (at 88.315 60 45) (layer F.SilkS)
+    (effects (font (size 1.2 1.2) (thickness 0.2)) (justify left))
+  )
+  (gr_line (start 82.55 103.505) (end 82.55 87.63) (layer F.SilkS) (width 0.12))
+  (gr_line (start 90.17 103.505) (end 82.55 103.505) (layer F.SilkS) (width 0.12))
+  (gr_line (start 90.17 87.63) (end 90.17 103.505) (layer F.SilkS) (width 0.12))
+  (gr_line (start 82.55 87.63) (end 90.17 87.63) (layer F.SilkS) (width 0.12))
+  (gr_text GND (at 85.725 88.9) (layer F.SilkS)
+    (effects (font (size 1 1) (thickness 0.15)))
+  )
+  (gr_text +12V (at 85.725 102.235) (layer F.SilkS)
+    (effects (font (size 1 1) (thickness 0.15)))
+  )
+  (gr_line (start 106.205 91.5) (end 102.235 91.44) (layer F.SilkS) (width 0.12))
+  (gr_line (start 102.235 60.96) (end 102.235 91.44) (layer F.SilkS) (width 0.12))
+  (gr_line (start 108.775 60.9) (end 102.235 60.96) (layer F.SilkS) (width 0.12))
+  (gr_text GND (at 106.045 90.17) (layer F.SilkS)
     (effects (font (size 1 1) (thickness 0.15)) (justify right))
   )
-  (gr_text SCL (at 105.41 87.63) (layer F.SilkS)
+  (gr_text SCL (at 105.902143 87.63) (layer F.SilkS)
     (effects (font (size 1 1) (thickness 0.15)) (justify right))
   )
-  (gr_text SDA (at 105.41 85.09) (layer F.SilkS)
+  (gr_text SDA (at 105.925952 85.09) (layer F.SilkS)
     (effects (font (size 1 1) (thickness 0.15)) (justify right))
   )
-  (gr_text IRQ (at 105.41 82.55) (layer F.SilkS)
+  (gr_text IRQ (at 105.783095 82.55) (layer F.SilkS)
     (effects (font (size 1 1) (thickness 0.15)) (justify right))
   )
-  (gr_text TRG (at 105.41 80.01) (layer F.SilkS)
+  (gr_text TRG (at 105.902143 80.01) (layer F.SilkS)
     (effects (font (size 1 1) (thickness 0.15)) (justify right))
   )
-  (gr_text 3V3 (at 105.41 77.47) (layer F.SilkS)
+  (gr_text 3V3 (at 105.902143 77.47) (layer F.SilkS)
     (effects (font (size 1 1) (thickness 0.15)) (justify right))
   )
-  (gr_text GND (at 105.41 74.93) (layer F.SilkS)
+  (gr_text GND (at 106.045 74.93) (layer F.SilkS)
     (effects (font (size 1 1) (thickness 0.15)) (justify right))
   )
-  (gr_text 5V (at 105.41 72.39) (layer F.SilkS)
+  (gr_text 5V (at 105.425952 72.39) (layer F.SilkS)
     (effects (font (size 1 1) (thickness 0.15)) (justify right))
   )
-  (gr_text GND (at 105.41 69.85) (layer F.SilkS)
+  (gr_text GND (at 106.045 69.85) (layer F.SilkS)
     (effects (font (size 1 1) (thickness 0.15)) (justify right))
   )
-  (gr_text 12V (at 105.41 67.31) (layer F.SilkS)
+  (gr_text 12V (at 105.902143 67.31) (layer F.SilkS)
     (effects (font (size 1 1) (thickness 0.15)) (justify right))
   )
-  (gr_text 12V (at 105.41 64.77) (layer F.SilkS)
+  (gr_text 12V (at 105.902143 64.77) (layer F.SilkS)
     (effects (font (size 1 1) (thickness 0.15)) (justify right))
   )
-  (gr_text GND (at 105.41 62.23) (layer F.SilkS)
+  (gr_text GND (at 106.045 62.23) (layer F.SilkS)
     (effects (font (size 1 1) (thickness 0.15)) (justify right))
   )
@@
   (segment (start 107.345 77.5) (end 107.315 77.47) (width 1.2) (layer F.Cu) (net 5))
   (segment (start 108.5 77.5) (end 107.345 77.5) (width 1.2) (layer F.Cu) (net 5))
-  (segment (start 109.775 101.85) (end 112 99.625) (width 1.2) (layer F.Cu) (net 5))
   (segment (start 112 81) (end 108.5 77.5) (width 1.2) (layer F.Cu) (net 5))
-  (segment (start 109.775 106) (end 109.775 101.85) (width 1.2) (layer F.Cu) (net 5))
   (segment (start 109.5 114.3) (end 109.5 111) (width 1.2) (layer F.Cu) (net 5))
   (segment (start 108.8 115) (end 109.5 114.3) (width 1.2) (layer F.Cu) (net 5))
@@
   (segment (start 99.5 110.5) (end 102.999992 110.5) (width 0.6) (layer B.Cu) (net 5))
   (segment (start 98.5 109.5) (end 99.5 110.5) (width 0.6) (layer B.Cu) (net 5))
-  (segment (start 112 99.625) (end 112 93.5) (width 1.2) (layer F.Cu) (net 5))
   (segment (start 112 84) (end 112 81) (width 1.2) (layer F.Cu) (net 5))
   (segment (start 112 93.5) (end 112 84) (width 1.2) (layer F.Cu) (net 5))
@@
   (segment (start 105.8125 93) (end 111.5 93) (width 0.4) (layer F.Cu) (net 5))
   (segment (start 101 88.1875) (end 105.8125 93) (width 0.4) (layer F.Cu) (net 5))
+  (segment (start 112 101.36) (end 112 93.5) (width 1.2) (layer F.Cu) (net 5))
+  (segment (start 109.775 103.585) (end 112 101.36) (width 1.2) (layer F.Cu) (net 5))
+  (segment (start 109.775 106) (end 109.775 103.585) (width 1.2) (layer F.Cu) (net 5))
   (segment (start 86.85556 75.10008) (end 87.455 75.69952) (width 0.4) (layer F.Cu) (net 6))
   (segment (start 86.60384 75.10008) (end 86.85556 75.10008) (width 0.4) (layer F.Cu) (net 6))

Commit message: WIP
Parts:
- removed C7: 220n, Capacitor_SMD:C_0805_2012Metric_Pad1.15x1.40mm_HandSolder
- added X1: SWD, Drake:SWD, F.Cu at (84.5, 65.0)
- C6: value 47M -> 100n; footprint Capacitor_SMD:C_0805_2012Metric_Pad1.15x1.40mm_HandSolder -> Capacitor_SMD:C_0805_2012Metric
- J1: footprint device.farm:DG301-5.0-02 -> Drake:DG301-5.0-02
- J2: footprint device.farm:conn_usb_B_micro_smd-2 -> Drake:conn_usb_B_micro_smd-2
- L1, L3: footprint device.farm:CKCS6028 -> Drake:CKCS6028
- U3: value MCP2221A -> ATSAMD11C14A-SS
- moved C8 7.83 mm to (88.0, 82.5), turned to 0 degrees
- moved C6 6.71 mm to (101.0, 79.5), turned to 90 degrees
- moved U3 3.54 mm to (94.5, 81.5), turned to 180 degrees
- moved R8 0.25 mm to (101.0, 87.5)
- turned DY1 to 270 degrees
Connections:
- C6 pad 1: Net-(C6-Pad1) -> GND
- C6 pad 2: GND -> Net-(C6-Pad2)
- C8 pad 2: Net-(C6-Pad1) -> +3V3
- DY1 pad 1: Net-(DY1-Pad1) -> GND
- DY1 pad 2: +3V3 -> Net-(DY1-Pad2)
- J2 pad 1: Net-(C6-Pad1) -> Net-(J2-Pad1)
- J2 pad 2: Net-(J2-Pad2) -> /USB_DM
- J2 pad 3: Net-(J2-Pad3) -> /USB_DP
- J2 pad 4: Net-(J2-Pad4) -> (no net)
- R4 pad 2: Net-(DY1-Pad1) -> Net-(DY1-Pad2)
- U3 pad 1: Net-(C6-Pad1) -> /IRQ
- U3 pad 10: /SCL -> /USB_DP
- U3 pad 11: Net-(C7-Pad1) -> GND
- U3 pad 12: Net-(J2-Pad2) -> +3V3
- U3 pad 13: Net-(J2-Pad3) -> /I2C_ACT
- U3 pad 14: GND -> /TRG
- U3 pad 2: /IRQ -> (no net)
- U3 pad 3: /TRG -> (no net)
- U3 pad 4: Net-(U3-Pad4) -> /SDA
- U3 pad 5: Net-(U3-Pad5) -> /SCL
- U3 pad 6: Net-(U3-Pad6) -> Net-(C6-Pad2)
- U3 pad 7: Net-(U3-Pad7) -> /SWCLK
- U3 pad 8: /I2C_ACT -> /SWDIO
- U3 pad 9: /SDA -> /USB_DM
Routing:
- net Net-(J2-Pad3): track 28.1 -> 0.00 mm
- net /SWCLK: track 0.00 -> 25.1 mm, vias 0 -> 2
- net /I2C_ACT: track 41.9 -> 18.0 mm, vias 2 -> 0
- net +3V3: track 124.4 -> 147.1 mm
- net Net-(J2-Pad2): track 21.8 -> 0.00 mm
- net Net-(C6-Pad1): track 16.1 -> 0.00 mm, vias 2 -> 0
- net /SWDIO: track 0.00 -> 14.7 mm
- net Net-(C7-Pad1): track 8.94 -> 0.00 mm
- net /USB_DP: track 0.00 -> 6.49 mm
- net /USB_DM: track 0.00 -> 6.24 mm
- net GND: track 43.9 -> 49.8 mm
- net /SCL: track 10.4 -> 15.6 mm
- net Net-(C6-Pad2): track 0.00 -> 4.19 mm
- net /TRG: track 39.6 -> 36.1 mm
- net Net-(DY1-Pad2): track 0.00 -> 2.04 mm
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Other:
- board text added: "SWD"
- board text added: "T100-USB v1.1"
- board text removed: "T100-USB v1"

Commit message: WIP
Parts:
- removed the DG1 at (99.5, 63.0)
- removed R14: 270R, Resistor_SMD:R_0805_2012Metric
- added C7: 100n, Capacitor_SMD:C_0805_2012Metric, F.Cu at (100.0, 75.0)
- DG1: renamed from DY1; value YELLOW -> GREEN
- J3: footprint Connector_PinSocket_2.54mm:PinSocket_1x12_P2.54mm_Horizontal -> Connector_PinSocket_2.54mm:PinSocket_1x10_P2.54mm_Horizontal
- R12: value 270R -> 1k5
- moved J3 5.08 mm to (107.3, 85.1)
- moved DR1 3.00 mm to (99.0, 63.0)
- moved R13 3.00 mm to (99.0, 67.0)
- moved DG1 1.50 mm to (94.0, 63.0)
- moved R4 1.50 mm to (94.0, 67.0)
- turned R10 to 90 degrees
- turned R11 to 90 degrees
Connections:
- net /TRG renamed /RST
- J3 pad 10: +12V -> GND
- J3 pad 7: GND -> +5V
- J3 pad 8: +5V -> +12V
- J3 pad 9: GND -> +12V
Routing:
- net /RST: track 36.1 -> 28.6 mm
- net +3V3: track 147.1 -> 140.1 mm
- net /SDA: track 29.6 -> 33.4 mm
- net +5V: track 82.9 -> 85.7 mm
- net GND: track 49.8 -> 47.7 mm, vias 18 -> 19
- net /IRQ: track 36.3 -> 38.4 mm
- net Net-(DG1-Pad1): track 2.04 -> 0.00 mm
- net /I2C_ACT: track 18.0 -> 18.8 mm
Other:
- board text added: "RST"
- board text removed: "TRG"
- board text removed: "trg"

Commit message: WIP
Parts:
- J1: footprint Drake:DG301-5.0-02 -> Drake:DG235-3.81-02P
- moved J1 5.02 mm to (91.0, 93.5)
- moved C1 1.50 mm to (95.0, 116.5)
- moved C2 1.50 mm to (92.0, 106.5)
- moved C3 1.50 mm to (96.0, 102.5)
- moved C5 1.50 mm to (106.0, 116.5)
- moved L1 1.50 mm to (107.0, 107.5)
- moved R1 1.50 mm to (100.0, 108.5)
- moved R2 1.50 mm to (96.0, 110.5)
- moved R3 1.50 mm to (92.0, 110.5)
- moved U2 1.50 mm to (96.0, 106.5)
Connections:
- J2 pad 1: Net-(J2-Pad1) -> unconnected-(J2-Pad1)
- J2 pad 4: (no net) -> unconnected-(J2-Pad4)
- U3 pad 2: (no net) -> unconnected-(U3-Pad2)
- U3 pad 3: (no net) -> unconnected-(U3-Pad3)
Routing:
- net +12V: track 226.1 -> 231.8 mm
- net +3V3: track 140.1 -> 141.5 mm
- net unconnected-(J2-Pad1): track 0.00 -> 1.10 mm
- net Net-(J2-Pad1): track 1.10 -> 0.00 mm
Other:
- net class Default removed

Commit message: WIP
Parts:
- removed C11, C18, C6, C7, C8: 100n, Capacitor_SMD:C_0805_2012Metric
- removed C19, C4, C5: 100u/12V, Capacitor_SMD:CP_Elec_6.3x5.4
- removed DG1: GREEN, LED_SMD:LED_0805_2012Metric_Pad1.15x1.40mm_HandSolder
- removed DR1: RED, LED_SMD:LED_0805_2012Metric_Pad1.15x1.40mm_HandSolder
- removed DW1: WHITE, LED_SMD:LED_0805_2012Metric_Pad1.15x1.40mm_HandSolder
- removed L1, L3: 6.8uH, Drake:CKCS6028
- removed R10, R11, R8, R9: 1K5, Resistor_SMD:R_0805_2012Metric
- removed R12: 1k5, Resistor_SMD:R_0805_2012Metric
- removed R13: 270R, Resistor_SMD:R_0805_2012Metric
- removed R7: 4.22k 1%, Resistor_SMD:R_0805_2012Metric
- removed U2: FR8205, Package_TO_SOT_SMD:SOT-23-6
- removed U3: ATSAMD11C14A-SS, Package_SO:SOIC-14_3.9x8.7mm_P1.27mm
- removed X1: SWD, Drake:SWD
- added D1: GREEN, LED_SMD:LED_0805_2012Metric_Pad1.15x1.40mm_HandSolder, F.Cu at (216.0, 68.0)
- added D2: RED, LED_SMD:LED_0805_2012Metric_Pad1.15x1.40mm_HandSolder, F.Cu at (220.8, 68.0)
- C1: value 100u/12V -> 100n; footprint Capacitor_SMD:CP_Elec_6.3x5.4 -> Capacitor_SMD:C_0805_2012Metric
- J1: value Conn_01x02_Female -> USB_B_Micro; footprint Drake:DG235-3.81-02P -> Drake:conn_usb_B_micro_smd-2
- J2: value USB_B_Micro -> T100-IN; footprint Drake:conn_usb_B_micro_smd-2 -> Connector_PinHeader_2.54mm:PinHeader_1x10_P2.54mm_Horizontal
- R1: value 100k -> 1K5
- R2: value 30k 1% -> 1K5
- R3: value 6.65k 1% -> 1K5
- R4: value 270R -> 1K5
- R5: value 100k -> 270R
- R6: value 30.9k 1% -> 270R
- U1: value FR8205 -> ATSAMD11C14A-SS; footprint Package_TO_SOT_SMD:SOT-23-6 -> Package_SO:SOIC-14_3.9x8.7mm_P1.27mm
- moved R5 146.7 mm to (221.4, 46.7), turned to 0 degrees
- moved R4 144.8 mm to (236.2, 39.5), turned to 0 degrees
- moved C2 138.5 mm to (217.0, 46.7), turned to 0 degrees
- moved R3 136.5 mm to (216.9, 55.6)
- moved R1 134.9 mm to (221.4, 49.6), turned to 0 degrees
- moved R2 134.0 mm to (216.9, 52.7)
- moved C3 132.0 mm to (217.0, 49.7)
- moved R6 129.4 mm to (208.4, 66.9)
- moved C1 111.6 mm to (195.0, 67.0)
- moved J1 83.1 mm to (152.0, 150.0), turned to 0 degrees
- moved J2 63.3 mm to (147.0, 86.9), turned to 180 degrees
- moved U1 57.7 mm to (153.0, 118.0), turned to -90 degrees
- moved J3 44.7 mm to (152.0, 86.9)
Connections:
- C1 pad 1: +12V -> GND
- C1 pad 2: GND -> +3V3
- C2 pad 2: +12V -> Net-(C2-Pad2)
- C3 pad 1: Net-(C3-Pad1) -> GND
- C3 pad 2: Net-(C3-Pad2) -> /RST
- J1 pad 1: GND -> unconnected-(J1-Pad1)
- J1 pad 2: +12V -> /USB_DM
- J2 pad 1: unconnected-(J2-Pad1) -> GND
- J2 pad 2: /USB_DM -> /SCL
- J2 pad 3: /USB_DP -> /SDA
- J2 pad 4: unconnected-(J2-Pad4) -> /IRQ
- J2 pad 5: GND -> /RST
- J2 pad 6: GND -> +3V3
- R1 pad 1: Net-(R1-Pad1) -> /SCL
- R1 pad 2: +12V -> +3V3
- R2 pad 1: Net-(R2-Pad1) -> /SDA
- R3 pad 1: GND -> /IRQ
- R3 pad 2: Net-(R2-Pad1) -> +3V3
- R4 pad 1: /I2C_ACT -> /RST
- R4 pad 2: Net-(DG1-Pad2) -> +3V3
- R5 pad 1: Net-(R5-Pad1) -> /I2C_ACT
- R5 pad 2: +12V -> Net-(D1-Pad2)
- R6 pad 1: Net-(R6-Pad1) -> /IRQ
- R6 pad 2: +5V -> Net-(D2-Pad1)
- U1 pad 1: Net-(C18-Pad1) -> /IRQ
- U1 pad 2: GND -> unconnected-(U1-Pad2)
- U1 pad 3: Net-(R6-Pad1) -> unconnected-(U1-Pad3)
- U1 pad 4: Net-(R5-Pad1) -> /SDA
- U1 pad 5: +12V -> /SCL
- U1 pad 6: Net-(C18-Pad2) -> Net-(C2-Pad2)
Routing:
- net +12V: track 231.8 -> 0.00 mm
- net +3V3: track 141.5 -> 0.00 mm, vias 2 -> 0
- net +5V: track 85.7 -> 0.00 mm, vias 2 -> 0
- net GND: track 47.7 -> 0.00 mm, vias 19 -> 0
- net /IRQ: track 38.3 -> 0.00 mm
- net /SDA: track 33.4 -> 0.00 mm
- net /RST: track 28.6 -> 0.00 mm, vias 2 -> 0
- net /SWCLK: track 25.1 -> 0.00 mm, vias 2 -> 0
- net /I2C_ACT: track 18.5 -> 0.00 mm
- net /SCL: track 16.0 -> 0.00 mm
- net /SWDIO: track 14.7 -> 0.00 mm
- net Net-(C18-Pad2): track 13.5 -> 0.00 mm
- net Net-(C3-Pad2): track 12.1 -> 0.00 mm
- net /USB_DP: track 6.49 -> 0.00 mm
- net /USB_DM: track 6.24 -> 0.00 mm
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- removed copper zone on B.Cu, net GND
Other:
- board size 34.5 x 99.5 mm -> 20 x 100 mm
- rule pad_to_mask_clearance: 0.051 -> 0
- board text removed: "+12V"
- board text removed: "12V"
- board text removed: "3V3"
- board text removed: "5V"
- board text removed: "GND"
- board text removed: "IRQ"
- board text removed: "RST"
- board text removed: "SCL"
- board text removed: "SDA"
- board text removed: "SWD"
- board text removed: "T100-USB v1.1"
- board text removed: "act"
- board text removed: "irq"
- board text removed: "pwr"

Commit message: WIP
Parts:
- moved R4 97.2 mm to (155.0, 93.0), turned to -90 degrees
- moved R5 95.3 mm to (146.0, 105.0), turned to 90 degrees
- moved C2 92.8 mm to (150.0, 111.0), turned to -90 degrees
- moved R1 87.0 mm to (146.0, 93.0), turned to -90 degrees
- moved R2 79.0 mm to (149.0, 93.0), turned to -90 degrees
- moved D1 77.4 mm to (146.0, 101.0), turned to -90 degrees
- moved R3 74.9 mm to (152.0, 93.0), turned to -90 degrees
- moved C3 73.1 mm to (158.0, 93.0), turned to 90 degrees
- moved D2 70.9 mm to (158.0, 101.0), turned to 90 degrees
- moved C1 70.2 mm to (154.0, 124.0)
- moved R6 63.2 mm to (158.0, 105.0), turned to 90 degrees
Routing:
- net +3V3: track 0.00 -> 89.6 mm
- net /RST: track 0.00 -> 57.5 mm, vias 0 -> 2
- net /IRQ: track 0.00 -> 49.2 mm, vias 0 -> 2
- net /SDA: track 0.00 -> 43.3 mm, vias 0 -> 2
- net /SCL: track 0.00 -> 42.7 mm
- net /USB_DM: track 0.00 -> 30.6 mm
- net /USB_DP: track 0.00 -> 30.6 mm
- net GND: track 0.00 -> 24.7 mm, vias 0 -> 6
- net /I2C_ACT: track 0.00 -> 22.2 mm
- net +12V: track 0.00 -> 15.1 mm
- net +5V: track 0.00 -> 5.00 mm
- net Net-(C2-Pad2): track 0.00 -> 3.77 mm
- net Net-(D2-Pad1): track 0.00 -> 2.06 mm
- net Net-(D1-Pad2): track 0.00 -> 2.06 mm
- net unconnected-(J1-Pad1): track 0.00 -> 1.10 mm
- added copper zone on B.Cu, net GND
Other:
- board text added: "ACT"
- board text added: "IRQ"
- board text added: "T100-USB v2.0"
