File: t100-usb/board/t100-usb.kicad_pcb (KiCad board)
At the start: 2 copper layers, 20 x 100 mm, 15 parts, among them J1 USB_B_Micro, J2 T100-IN, J3 T100-OUT, U1 ATSAMD11C14A-SS

Commit message: WIP
Routing:
- net GND: track 24.7 -> 29.7 mm
- net /IRQ: track 49.2 -> 48.6 mm
Changed lines of the file:
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@@
   (segment (start 153 123.95) (end 153.05 124) (width 0.4) (layer "F.Cu") (net 1))
   (segment (start 153.05 125.95) (end 153.05 124) (width 0.4) (layer "F.Cu") (net 1))
+  (segment (start 147 64) (end 152 64) (width 2) (layer "F.Cu") (net 1))
   (via (at 146 98) (size 0.8) (drill 0.4) (layers "F.Cu" "B.Cu") (net 1))
   (via (at 146 150) (size 0.8) (drill 0.4) (layers "F.Cu" "B.Cu") (net 1))
@@
   (segment (start 154.27 123.32) (end 154.95 124) (width 0.4) (layer "F.Cu") (net 2))
   (segment (start 154.27 120.475) (end 154.27 123.32) (width 0.4) (layer "F.Cu") (net 2))
+  (segment (start 152 74.16) (end 147 74.16) (width 2) (layer "F.Cu") (net 2))
   (segment (start 160.975 99.975) (end 161 100) (width 0.4) (layer "F.Cu") (net 2))
   (segment (start 158.16 74.16) (end 161 77) (width 0.4) (layer "F.Cu") (net 2))
@@
   (segment (start 146 93.9125) (end 155 93.9125) (width 0.4) (layer "F.Cu") (net 2))
   (segment (start 161 121) (end 158 124) (width 0.4) (layer "F.Cu") (net 2))
-  (segment (start 147 74.16) (end 152 74.16) (width 2) (layer "B.Cu") (net 2))
   (segment (start 150.46 115.525) (end 150.46 112.41) (width 0.4) (layer "F.Cu") (net 3))
   (segment (start 150.46 112.41) (end 150 111.95) (width 0.4) (layer "F.Cu") (net 3))
+  (segment (start 152 76.7) (end 147 76.7) (width 2) (layer "F.Cu") (net 4))
   (segment (start 155 92.0875) (end 154.5 91.5875) (width 0.4) (layer "F.Cu") (net 4))
   (segment (start 159.05 120.475) (end 156.81 120.475) (width 0.4) (layer "F.Cu") (net 4))
@@
   (via (at 160 98) (size 0.8) (drill 0.4) (layers "F.Cu" "B.Cu") (net 4))
   (segment (start 160 108.5) (end 160 98) (width 0.4) (layer "B.Cu") (net 4))
-  (segment (start 152 76.7) (end 147 76.7) (width 2) (layer "B.Cu") (net 4))
   (segment (start 150.10008 147.59944) (end 150.69952 147) (width 0.4) (layer "F.Cu") (net 5))
   (segment (start 150.10008 147.85116) (end 150.10008 147.59944) (width 0.4) (layer "F.Cu") (net 5))
@@
   (segment (start 149 96) (end 149 90) (width 0.4) (layer "B.Cu") (net 10))
   (segment (start 156.9125 105.9125) (end 155 104) (width 0.4) (layer "F.Cu") (net 11))
+  (segment (start 152 90) (end 151 90) (width 0.4) (layer "F.Cu") (net 11))
   (segment (start 155 104) (end 155 99) (width 0.4) (layer "F.Cu") (net 11))
-  (segment (start 150 81.24) (end 152 79.24) (width 0.4) (layer "F.Cu") (net 11))
   (segment (start 152 92.0875) (end 152 90) (width 0.4) (layer "F.Cu") (net 11))
+  (segment (start 151 90) (end 150 89) (width 0.4) (layer "F.Cu") (net 11))
   (segment (start 155 99) (end 152 96) (width 0.4) (layer "F.Cu") (net 11))
   (segment (start 158 105.9125) (end 158 114.335) (width 0.4) (layer "F.Cu") (net 11))
-  (segment (start 152 90) (end 151 90) (width 0.4) (layer "F.Cu") (net 11))
   (segment (start 158 105.9125) (end 156.9125 105.9125) (width 0.4) (layer "F.Cu") (net 11))
-  (segment (start 150 89) (end 150 81.24) (width 0.4) (layer "F.Cu") (net 11))
-  (segment (start 151 90) (end 150 89) (width 0.4) (layer "F.Cu") (net 11))
+  (segment (start 152 79.24) (end 147 79.24) (width 2) (layer "F.Cu") (net 11))
+  (segment (start 150 89) (end 150 79) (width 0.4) (layer "F.Cu") (net 11))
   (segment (start 158 114.335) (end 156.81 115.525) (width 0.4) (layer "F.Cu") (net 11))
   (via (at 152 90) (size 0.8) (drill 0.4) (layers "F.Cu" "B.Cu") (net 11))
   (via (at 152 96) (size 0.8) (drill 0.4) (layers "F.Cu" "B.Cu") (net 11))
-  (segment (start 147 79.24) (end 152 79.24) (width 2) (layer "B.Cu") (net 11))
   (segment (start 152 96) (end 152 90) (width 0.4) (layer "B.Cu") (net 11))
-  (segment (start 147 71.62) (end 152 71.62) (width 2) (layer "B.Cu") (net 12))
-  (segment (start 152 66.54) (end 152 69.08) (width 2) (layer "B.Cu") (net 13))
-  (segment (start 152 66.54) (end 147 66.54) (width 2) (layer "B.Cu") (net 13))
-  (segment (start 147 66.54) (end 147 69.08) (width 2) (layer "B.Cu") (net 13))
-  (segment (start 147 69.08) (end 152 69.08) (width 2) (layer "B.Cu") (net 13))
+  (segment (start 152 71.62) (end 147 71.62) (width 2) (layer "F.Cu") (net 12))
+  (segment (start 152 69.08) (end 152 66.54) (width 2) (layer "F.Cu") (net 13))
+  (segment (start 147 69.08) (end 152 69.08) (width 2) (layer "F.Cu") (net 13))
+  (segment (start 152 66.54) (end 147 66.54) (width 2) (layer "F.Cu") (net 13))
+  (segment (start 147 66.54) (end 147 69.08) (width 2) (layer "F.Cu") (net 13))
   (segment (start 146 116) (end 146 105.9125) (width 0.4) (layer "F.Cu") (net 14))
   (segment (start 155.54 119.266431) (end 154.273569 118) (width 0.4) (layer "F.Cu") (net 14))
