File: t100-dcmotor/board/t100-dcmotor.kicad_pcb (KiCad board)
At the start: 2 copper layers, 34.5 x 99.5 mm, 29 parts, among them J1 T100-IN, J2 T100-OUT, J3 Conn_01x08_Female, U1 ATSAMD11D14A-SS, U2 VNH7070BAS, X1 SWD

Commit message: WIP
Other:
- board text added: "12V DC MOTOR DRIVER W/ HALL ENCODER v1"
- board text removed: "12V DC MOTOR DRIVER W/ HALL ENCODER"
Changed lines of the file:
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@@
     (solder_mask_min_width 0.25)
     (aux_axis_origin 0 0)
-    (grid_origin 87.5 124.5)
     (visible_elements FFFFFF7F)
     (pcbplotparams
@@
     (arrow2b (pts (xy 82.5 40) (xy 83.626504 39.413579)))
   )
-  (gr_text "12V DC MOTOR DRIVER\nW/ HALL ENCODER" (at 100 55) (layer F.SilkS)
-    (effects (font (size 1 1) (thickness 0.15)))
+  (gr_text "12V DC MOTOR DRIVER\nW/ HALL ENCODER v1" (at 100 55) (layer F.SilkS)
+    (effects (font (size 1 1) (thickness 0.2)))
   )
   (gr_arc (start 87.5 145) (end 87.5 146.75) (angle -180) (layer Edge.Cuts) (width 0.254))

Commit message: WIP
Parts:
- J3: footprint device.farm:DG235-3.81-08P -> Drake:DG235-3.81-08P
- X1: footprint device.farm:SWD -> Drake:SWD
Changed lines of the file:
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@@
     )
   )
-  (module device.farm:DG235-3.81-08P (layer F.Cu)
+  (module Drake:DG235-3.81-08P (layer F.Cu)
     (at 87.5 124.5)
     (fp_text reference J3 (at 0 -4) (layer F.SilkS)
@@
     (pad 8 thru_hole roundrect (at 26.67 0) (size 2.2 2.2) (drill 1.2) (layers *.Cu *.Mask) (roundrect_rratio 0.25)
       (net 31 /STOP_2))
-    (model ${DF_3D}/DG235-3.81-08P.step
+    (model ${HW_KICAD}/footprints/DG235-3.81-08P.step
       (at (xyz 0 0 0))
       (scale (xyz 1 1 1))
@@
     )
   )
-  (module device.farm:SWD (layer F.Cu)
+  (module Drake:SWD (layer F.Cu)
     (at 101.5 96.5 270)
     (fp_text reference X1 (at -3 -2.5 90) (layer F.SilkS) hide

Commit message: WIP
Parts:
- removed R12: A-270R B-N/A Z-10k, Resistor_SMD:R_0805_2012Metric_Pad1.15x1.40mm_HandSolder
- removed R13: A-N/A B-270R Z-10k, Resistor_SMD:R_0805_2012Metric_Pad1.15x1.40mm_HandSolder
- removed R5: 1k, Resistor_SMD:R_0805_2012Metric_Pad1.15x1.40mm_HandSolder
- added D4: BAT54S, Package_TO_SOT_SMD:SOT-23, F.Cu at (90.0, 95.5)
- added JP1: SolderJumper_3_Open, Jumper:SolderJumper-3_P2.0mm_Open_TrianglePad1.0x1.5mm, F.Cu at (103.5, 66.5)
- added ST1: SolderJumper_2_Open, Jumper:SolderJumper-2_P1.3mm_Open_TrianglePad1.0x1.5mm, F.Cu at (114.5, 116.5)
- added ST2: SolderJumper_2_Open, Jumper:SolderJumper-2_P1.3mm_Open_TrianglePad1.0x1.5mm, F.Cu at (114.5, 119.5)
- C2: value 10n -> 1u
- J1: footprint Connector_PinHeader_2.54mm:PinHeader_1x12_P2.54mm_Horizontal -> Connector_PinHeader_2.54mm:PinHeader_1x10_P2.54mm_Horizontal
- J2: footprint Connector_PinSocket_2.54mm:PinSocket_1x12_P2.54mm_Horizontal -> Connector_PinSocket_2.54mm:PinSocket_1x10_P2.54mm_Horizontal
- R2, R3, R4: value 1k -> 1k5
- R9: value (sense?) -> 1k5
- moved J1 5.08 mm to (87.8, 85.1)
- moved J2 5.08 mm to (107.2, 85.1)
Connections:
- J1 pad 10: +12V -> GND
- J1 pad 5: /TRG -> /RST
- J1 pad 7: GND -> +5V
- J1 pad 8: +5V -> +12V
- J1 pad 9: GND -> +12V
- J2 pad 10: +12V -> GND
- J2 pad 5: /TRG -> /RST
- J2 pad 7: GND -> +5V
- J2 pad 8: +5V -> +12V
- J2 pad 9: GND -> +12V
- U1 pad 1: /IRQ -> /STOP_2
- U1 pad 10: /SEL0 -> /IRQ
- U1 pad 11: Net-(U1-Pad11) -> /RST
- U1 pad 20: /TRG -> /STOP_1
- U1 pad 4: /STOP_1 -> (no net)
- U1 pad 5: /STOP_2 -> (no net)
- U2 pad 14: Net-(R5-Pad1) -> Net-(R2-Pad1)
Routing:
- net GND: track 115.1 -> 68.8 mm, vias 31 -> 32
- net /RST: track 0.00 -> 42.8 mm, vias 0 -> 2
- net Net-(R5-Pad1): track 32.1 -> 0.00 mm, vias 2 -> 0
- net /TRG: track 25.4 -> 0.00 mm
- net /IRQ: track 24.2 -> 36.1 mm
- net /SEL0: track 11.2 -> 0.00 mm
- net /ADDR: track 28.2 -> 17.8 mm
- net /STOP_1: track 117.5 -> 124.3 mm, vias 1 -> 4
- net +3V3: track 159.2 -> 164.5 mm, vias 0 -> 2
- net Net-(R2-Pad1): track 19.1 -> 24.3 mm
- net /HALL_B: track 38.8 -> 42.5 mm
- net /SDA: track 24.3 -> 27.6 mm
- net +5V: track 48.6 -> 51.1 mm
- net /SCL: track 24.4 -> 26.8 mm
- net /CS: track 30.6 -> 28.4 mm, vias 2 -> 0
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Other:
- board text added: "12V DC MOTOR DRIVER W/ HALL ENCODER v1.1"
- board text added: "A"
- board text added: "B"
- board text removed: "12V DC MOTOR DRIVER W/ HALL ENCODER v1"

Commit message: WIP
Parts:
- removed D4: BAT54S, Package_TO_SOT_SMD:SOT-23
- removed R4, R9: 1k5, Resistor_SMD:R_0805_2012Metric_Pad1.15x1.40mm_HandSolder
- removed R6: 10k, Resistor_SMD:R_0805_2012Metric_Pad1.15x1.40mm_HandSolder
- added C5: 10u, Capacitor_SMD:C_0805_2012Metric_Pad1.18x1.45mm_HandSolder, F.Cu at (95.5, 115.5)
- C1: footprint Capacitor_SMD:C_0805_2012Metric_Pad1.15x1.40mm_HandSolder -> Capacitor_SMD:C_0805_2012Metric_Pad1.18x1.45mm_HandSolder
- C2: value 1u -> 100n; footprint Capacitor_SMD:C_0805_2012Metric_Pad1.15x1.40mm_HandSolder -> Capacitor_SMD:C_0805_2012Metric_Pad1.18x1.45mm_HandSolder
- C3: value 100n -> 10u; footprint Capacitor_SMD:C_0805_2012Metric_Pad1.15x1.40mm_HandSolder -> Capacitor_SMD:C_0805_2012Metric_Pad1.18x1.45mm_HandSolder
- C4: value 270p -> 10u; footprint Capacitor_SMD:C_0805_2012Metric_Pad1.15x1.40mm_HandSolder -> Capacitor_SMD:C_0805_2012Metric_Pad1.18x1.45mm_HandSolder
- R1, R10, R11, R14, R15, R2, R3, R7, R8: footprint Resistor_SMD:R_0805_2012Metric_Pad1.15x1.40mm_HandSolder -> Resistor_SMD:R_0805_2012Metric_Pad1.20x1.40mm_HandSolder
- U2: value VNH7070BAS -> ZXBM5210-SP; footprint Package_SO:SOIC-16_3.9x9.9mm_P1.27mm -> Package_SO:Diodes_SO-8EP
- moved C4 17.0 mm to (89.5, 115.5), turned to 0 degrees
- moved C2 11.9 mm to (88.5, 108.0), turned to 180 degrees
- moved R2 8.02 mm to (90.0, 95.0)
- moved R3 7.83 mm to (92.5, 95.0)
- moved C3 6.58 mm to (100.5, 108.5), turned to 90 degrees
- moved U2 6.40 mm to (95.0, 110.0), turned to 180 degrees
- moved R10 1.50 mm to (85.0, 112.5)
- moved X1 1.50 mm to (101.5, 98.0)
Connections:
- C2 pad 1: /CS -> +3V3
- C4 pad 1: +12V -> /MOTOR_M
- R2 pad 2: /INA -> /FWD
- R3 pad 2: /INB -> /REV
- U1 pad 14: /INA -> /LED
- U1 pad 15: /INB -> (no net)
- U1 pad 18: /CS -> (no net)
- U1 pad 8: /PWM -> /FWD
- U1 pad 9: /LED -> /REV
- U2 pad 1: GND -> /MOTOR_P
- U2 pad 2: /MOTOR_P -> +12V
- U2 pad 3: Net-(R2-Pad1) -> +3V3
- U2 pad 4: +12V -> Net-(R2-Pad1)
- U2 pad 5: +12V -> Net-(R3-Pad1)
- U2 pad 6: Net-(R3-Pad1) -> +3V3
Routing:
- net Net-(R6-Pad1): track 29.6 -> 0.00 mm, vias 2 -> 0
- net /CS: track 28.4 -> 0.00 mm
- net +3V3: track 164.5 -> 186.4 mm, vias 2 -> 0
- net /PWM: track 21.7 -> 0.00 mm
- net GND: track 68.8 -> 90.4 mm, vias 32 -> 17
- net Net-(R4-Pad1): track 19.6 -> 0.00 mm, vias 2 -> 0
- net /INB: track 18.4 -> 0.00 mm
- net +12V: track 107.4 -> 96.7 mm
- net /INA: track 8.99 -> 0.00 mm
- net /MOTOR_M: track 28.1 -> 19.5 mm
- net /FWD: track 0.00 -> 7.40 mm
- net /REV: track 0.00 -> 6.54 mm
- net Net-(R2-Pad1): track 24.3 -> 19.9 mm
- net /LED: track 18.7 -> 14.4 mm
- net /MOTOR_P: track 27.3 -> 23.5 mm
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- added copper zone on F.Cu, net +12V
- added copper zone on F.Cu, net /MOTOR_M
- removed copper zone on F.Cu, net GND
