File: t100-dcmotor/board/t100-dcmotor.sch (KiCad schematic (older format))
At the start: 29 parts, among them J1 T100-IN, J2 T100-OUT, J3 Conn_01x08_Female, U1 ATSAMD11D14A-SS, U2 VNH7070BAS, X1 SWD

Commit message: WIP
Parts:
- J1: symbol device.farm:T100-IN -> Drake:T100-IN
- J2: symbol device.farm:T100-OUT -> Drake:T100-OUT
- J3: footprint device.farm:DG235-3.81-08P -> Drake:DG235-3.81-08P
- U2: symbol device.farm:VNH7070BAS -> Drake:VNH7070BAS
- X1: footprint device.farm:SWD -> Drake:SWD; symbol device.farm:SWD -> Drake:SWD
Changed lines of the file:
@@
 $EndDescr
 $Comp
-L device.farm:T100-IN J1
+L Drake:T100-IN J1
 U 1 1 6001E3D6
 P 1200 2300
@@
 $EndComp
 $Comp
-L device.farm:T100-OUT J2
+L Drake:T100-OUT J2
 U 1 1 6001E716
 P 2100 2250
@@
 TRG
 $Comp
-L device.farm:VNH7070BAS U2
+L Drake:VNH7070BAS U2
 U 1 1 600288BD
 P 9000 2250
@@
 HALL_B
 $Comp
-L device.farm:SWD X1
+L Drake:SWD X1
 U 1 1 60037E8A
 P 1500 4950
 F 0 "X1" H 1608 5297 60  0000 C CNN
 F 1 "SWD" H 1608 5191 60  0000 C CNN
-F 2 "device.farm:SWD" H 1500 4750 60  0001 C CNN
+F 2 "Drake:SWD" H 1500 4750 60  0001 C CNN
 F 3 "" H 1500 4950 60  0000 C CNN
 	1    1500 4950
@@
 F 0 "J3" H 9928 4976 50  0000 L CNN
 F 1 "Conn_01x08_Female" H 9928 4885 50  0000 L CNN
-F 2 "device.farm:DG235-3.81-08P" H 9900 5000 50  0001 C CNN
+F 2 "Drake:DG235-3.81-08P" H 9900 5000 50  0001 C CNN
 F 3 "~" H 9900 5000 50  0001 C CNN
 	1    9900 5000

Commit message: WIP
Parts:
- removed R12: A-270R B-N/A Z-10k, Resistor_SMD:R_0805_2012Metric_Pad1.15x1.40mm_HandSolder, symbol Device:R
- removed R13: A-N/A B-270R Z-10k, Resistor_SMD:R_0805_2012Metric_Pad1.15x1.40mm_HandSolder, symbol Device:R
- removed R5: 1k, Resistor_SMD:R_0805_2012Metric_Pad1.15x1.40mm_HandSolder, symbol Device:R
- added D4: BAT54S, Package_TO_SOT_SMD:SOT-23, symbol Diode:BAT54S
- added JP1: SolderJumper_3_Open, Jumper:SolderJumper-3_P2.0mm_Open_TrianglePad1.0x1.5mm, symbol Jumper:SolderJumper_3_Open
- added ST1, ST2: SolderJumper_2_Open, Jumper:SolderJumper-2_P1.3mm_Open_TrianglePad1.0x1.5mm, symbol Jumper:SolderJumper_2_Open
- C2: value 10n -> 1u
- FB1: symbol Device:Ferrite_Bead_Small -> Device:FerriteBead_Small
- J1: footprint Connector_PinHeader_2.54mm:PinHeader_1x12_P2.54mm_Horizontal -> Connector_PinHeader_2.54mm:PinHeader_1x10_P2.54mm_Horizontal
- J2: footprint Connector_PinSocket_2.54mm:PinSocket_1x12_P2.54mm_Horizontal -> Connector_PinSocket_2.54mm:PinSocket_1x10_P2.54mm_Horizontal
- R2, R3, R4: value 1k -> 1k5
- R9: value (sense?) -> 1k5
Connections:
- net labels added: RST
- net labels removed: SEL0, TRG
- wire segments 64 -> 59
- no-connect marks 1 -> 2
Other:
- note removed: "pullup k STOP1/2"
- note removed: "zmenit velikost R7, R8"
- moved on the sheet: J1, J2

Commit message: WIP
Parts:
- removed D4: BAT54S, Package_TO_SOT_SMD:SOT-23, symbol Diode:BAT54S
- removed R4, R9: 1k5, Resistor_SMD:R_0805_2012Metric_Pad1.15x1.40mm_HandSolder, symbol Device:R
- removed R6: 10k, Resistor_SMD:R_0805_2012Metric_Pad1.15x1.40mm_HandSolder, symbol Device:R
- removed U2: VNH7070BAS, Package_SO:SOIC-16_3.9x9.9mm_P1.27mm, symbol Drake:VNH7070BAS
- added C5: 10u, Capacitor_SMD:C_0805_2012Metric_Pad1.18x1.45mm_HandSolder, symbol Device:C
- added U2: ZXBM5210-SP, Package_SO:Diodes_SO-8EP, symbol Driver_Motor:ZXBM5210-SP
- C1: footprint Capacitor_SMD:C_0805_2012Metric_Pad1.15x1.40mm_HandSolder -> Capacitor_SMD:C_0805_2012Metric_Pad1.18x1.45mm_HandSolder
- C2: value 1u -> 100n; footprint Capacitor_SMD:C_0805_2012Metric_Pad1.15x1.40mm_HandSolder -> Capacitor_SMD:C_0805_2012Metric_Pad1.18x1.45mm_HandSolder
- C3: value 100n -> 10u; footprint Capacitor_SMD:C_0805_2012Metric_Pad1.15x1.40mm_HandSolder -> Capacitor_SMD:C_0805_2012Metric_Pad1.18x1.45mm_HandSolder
- C4: value 270p -> 10u; footprint Capacitor_SMD:C_0805_2012Metric_Pad1.15x1.40mm_HandSolder -> Capacitor_SMD:C_0805_2012Metric_Pad1.18x1.45mm_HandSolder
- R1, R10, R11, R14, R15, R2, R3, R7, R8: footprint Resistor_SMD:R_0805_2012Metric_Pad1.15x1.40mm_HandSolder -> Resistor_SMD:R_0805_2012Metric_Pad1.20x1.40mm_HandSolder
Connections:
- net PWM is gone; now on net FWD: U1.8 (PA16)
- net +12V: now also U2.2 (VM); no longer C4.1
- net +3V3: now also C2.1, U2.3 (VDD), U2.6 (VREF)
- net GND: now also C5.2, U2.8 (GND), U2.9 (GND)
- net LED: now also U1.14 (PA24); no longer U1.9 (PA22)
- net MOTOR_M: now also C4.1, U2.7 (OUT2)
- net MOTOR_P: now also C5.1, U2.1 (OUT1)
- net at R2.1: now also U2.4 (FWD)
- net at R3.1: now also U2.5 (REV)
- net CS: no longer names the net of U1.18 (PA02)
- net CS: no longer C2.1
- net INA renamed FWD
- net FWD: no longer U1.14 (PA24)
- net INB: no longer names the net of U1.15 (PA25)
- net INB: no longer R3.2
- new net REV: R3.2, U1.9 (PA22)
- no-connect marks 2 -> 4
Other:
- moved on the sheet: C3, R2, R3

Commit message: WIP
Parts:
- FB1: symbol Device:FerriteBead_Small -> Device:Ferrite_Bead_Small
- U2: footprint Package_SO:Diodes_SO-8EP -> Package_SO:SOIC-8-1EP_3.9x4.9mm_P1.27mm_EP2.41x3.3mm
Changed lines of the file:
@@
 $EndComp
 $Comp
-L Device:FerriteBead_Small FB1
+L Device:Ferrite_Bead_Small FB1
 U 1 1 601A6B45
 P 8000 5850
@@
 F 0 "U2" H 9400 2750 50  0000 C CNN
 F 1 "ZXBM5210-SP" H 9600 2650 50  0000 C CNN
-F 2 "Package_SO:Diodes_SO-8EP" H 9050 2000 50  0001 C CNN
+F 2 "Package_SO:SOIC-8-1EP_3.9x4.9mm_P1.27mm_EP2.41x3.3mm" H 9050 2000 50  0001 C CNN
 F 3 "https://www.diodes.com/assets/Datasheets/ZXBM5210.pdf" H 9000 2250 50  0001 C CNN
 	1    9000 2250
