File: t100-dcmotor/board/t100-dcmotor.kicad_sch (KiCad schematic)
At the start: 27 parts, among them J1 T100-IN, J2 T100-OUT, J3 Conn_01x08_Female, U1 ATSAMD11D14A-SS, U2 ZXBM5210-SP, X1 SWD

Commit message: WIP
Parts:
- removed C5: 10u, Capacitor_SMD:C_0805_2012Metric_Pad1.18x1.45mm_HandSolder, symbol Device:C
- removed R2, R3: 1k5, Resistor_SMD:R_0805_2012Metric_Pad1.20x1.40mm_HandSolder, symbol Device:R
- removed U2: ZXBM5210-SP, Package_SO:Diodes_SO-8EP, symbol Driver_Motor:ZXBM5210-SP
- added U2: TB67H451FNG, Package_SO:HSOP-8-1EP_3.9x4.9mm_P1.27mm_EP2.41x3.1mm, symbol Drake:TB67H451FNG
- C3: value 10u -> 100u/16V; footprint Capacitor_SMD:C_0805_2012Metric_Pad1.18x1.45mm_HandSolder -> Capacitor_SMD:CP_Elec_6.3x5.4; symbol Device:C -> Device:C_Polarized
- C4: value 10u -> 100n
Connections:
- net +12V: now also C2.1, U2.5 (VM)
- net +3V3: now also C4.1, U2.4 (VREF); no longer C2.1
- net GND: now also U2.1 (GND), U2.7 (RS), U2.9 (GND)
- net MOTOR_M: now also U2.6 (OUT1); no longer C4.1
- net MOTOR_P: now also U2.8 (OUT2)
- net FWD renamed MOTOR_1
- net MOTOR_1: now also U2.2 (IN1)
- net REV renamed MOTOR_2
- net MOTOR_2: now also U2.3 (IN2)
Other:
- moved on the sheet: C2

Commit message: WIP
Parts:
- removed R10, R11: 270R, Resistor_SMD:R_0805_2012Metric_Pad1.20x1.40mm_HandSolder, symbol Device:R
- added C? (x2): 100n, Capacitor_SMD:C_0805_2012Metric_Pad1.18x1.45mm_HandSolder, symbol Device:C
- R7, R8: value 10k -> 1k5
Connections:
- net GND: now also C?.1, C?.2
- net HALL_A: now also J3.4 (Pin_4), C?.1
- net HALL_B: now also J3.3 (Pin_3), C?.2

Commit message: WIP
Parts:
- removed C? (x2): 100n, Capacitor_SMD:C_0805_2012Metric_Pad1.18x1.45mm_HandSolder, symbol Device:C
- removed D2, D3: BAT54S, Package_TO_SOT_SMD:SOT-23, symbol Diode:BAT54S
- removed R14, R15: 10k, Resistor_SMD:R_0805_2012Metric_Pad1.20x1.40mm_HandSolder, symbol Device:R
- removed R7, R8: 1k5, Resistor_SMD:R_0805_2012Metric_Pad1.20x1.40mm_HandSolder, symbol Device:R
- renumbered C3 to C2, C4 to C3, C2 to C4
Connections:
- net HALL_A: no longer J3.4 (Pin_4)
- net HALL_B: no longer J3.3 (Pin_3)
- net STOP_1: no longer J3.7 (Pin_7)
- net STOP_2: no longer J3.8 (Pin_8)
- new net input-filter/PORT: J3.3 (Pin_3)
- new net input-filter1/PORT: J3.4 (Pin_4)
- new net input-filter2/PORT: J3.7 (Pin_7)
- new net input-filter3/PORT: J3.8 (Pin_8)
Other:
- added sheet input-filter (input-filter.kicad_sch)
- added sheet input-filter1 (input-filter.kicad_sch)
- added sheet input-filter2 (input-filter.kicad_sch)
- added sheet input-filter3 (input-filter.kicad_sch)
- moved on the sheet: FB1

Commit message: WIP
Parts:
- added R10: 0R47, Resistor_SMD:R_1206_3216Metric_Pad1.30x1.75mm_HandSolder, symbol Device:R
Connections:
- net GND: now also R10.1; no longer U2.7 (RS)
- new net: R10.2, U2.7 (RS)
Changed lines of the file:
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@@
   (junction (at 63.5 52.07) (diameter 0) (color 0 0 0 0)
   )
-  (junction (at 229.87 74.93) (diameter 0) (color 0 0 0 0)
+  (junction (at 229.87 83.82) (diameter 0) (color 0 0 0 0)
   )
   (no_connect (at 110.49 60.96))
@@
     (stroke (width 0) (type default) (color 0 0 0 0))
   )
+  (wire (pts (xy 232.41 81.28) (xy 232.41 83.82))
+    (stroke (width 0) (type default) (color 0 0 0 0))
+  )
   (wire (pts (xy 57.15 52.07) (xy 63.5 52.07))
     (stroke (width 0) (type default) (color 0 0 0 0))
   )
-  (wire (pts (xy 229.87 73.66) (xy 229.87 74.93))
+  (wire (pts (xy 232.41 83.82) (xy 229.87 83.82))
+    (stroke (width 0) (type default) (color 0 0 0 0))
+  )
+  (wire (pts (xy 229.87 73.66) (xy 229.87 83.82))
     (stroke (width 0) (type default) (color 0 0 0 0))
   )
@@
     (stroke (width 0) (type default) (color 0 0 0 0))
   )
-  (wire (pts (xy 232.41 73.66) (xy 232.41 74.93))
-    (stroke (width 0) (type default) (color 0 0 0 0))
-  )
-  (wire (pts (xy 232.41 74.93) (xy 229.87 74.93))
-    (stroke (width 0) (type default) (color 0 0 0 0))
-  )
   (wire (pts (xy 234.95 147.32) (xy 234.95 137.16))
     (stroke (width 0) (type default) (color 0 0 0 0))
@@
     (stroke (width 0) (type default) (color 0 0 0 0))
   )
-  (wire (pts (xy 227.33 73.66) (xy 227.33 74.93))
-    (stroke (width 0) (type default) (color 0 0 0 0))
-  )
-  (wire (pts (xy 227.33 74.93) (xy 229.87 74.93))
-    (stroke (width 0) (type default) (color 0 0 0 0))
-  )
-  (wire (pts (xy 229.87 74.93) (xy 229.87 76.2))
+  (wire (pts (xy 227.33 73.66) (xy 227.33 83.82))
+    (stroke (width 0) (type default) (color 0 0 0 0))
+  )
+  (wire (pts (xy 227.33 83.82) (xy 229.87 83.82))
+    (stroke (width 0) (type default) (color 0 0 0 0))
+  )
+  (wire (pts (xy 229.87 83.82) (xy 229.87 85.09))
     (stroke (width 0) (type default) (color 0 0 0 0))
   )
@@
     (pin "1")
   )
-  (symbol (lib_id "power:GND") (at 229.87 76.2 0) (unit 1)
-    (in_bom yes) (on_board yes)
-    (property "Reference" "#PWR023" (id 0) (at 229.87 82.55 0)
-      (effects (font (size 1.27 1.27)) hide)
-    )
-    (property "Value" "GND" (id 1) (at 229.997 80.5942 0))
-    (property "Footprint" "" (id 2) (at 229.87 76.2 0)
-      (effects (font (size 1.27 1.27)) hide)
-    )
-    (property "Datasheet" "" (id 3) (at 229.87 76.2 0)
+  (symbol (lib_id "power:GND") (at 229.87 85.09 0) (unit 1)
+    (in_bom yes) (on_board yes)
+    (property "Reference" "#PWR023" (id 0) (at 229.87 91.44 0)
+      (effects (font (size 1.27 1.27)) hide)
+    )
+    (property "Value" "GND" (id 1) (at 229.997 89.4842 0))
+    (property "Footprint" "" (id 2) (at 229.87 85.09 0)
+      (effects (font (size 1.27 1.27)) hide)
+    )
+    (property "Datasheet" "" (id 3) (at 229.87 85.09 0)
       (effects (font (size 1.27 1.27)) hide)
     )
@@
     (pin "1")
   )
+  (symbol (lib_id "Device:R") (at 232.41 77.47 180) (unit 1)
+    (in_bom yes) (on_board yes)
+    (property "Reference" "R10" (id 0) (at 237.6678 77.47 90))
+    (property "Value" "0R47" (id 1) (at 235.3564 77.47 90))
+    (property "Footprint" "Resistor_SMD:R_1206_3216Metric_Pad1.30x1.75mm_HandSolder" (id 2) (at 234.188 77.47 90)
+      (effects (font (size 1.27 1.27)) hide)
+    )
+    (property "Datasheet" "~" (id 3) (at 232.41 77.47 0)
+      (effects (font (size 1.27 1.27)) hide)
+    )
+    (pin "1")
+    (pin "2")
+  )
   (symbol (lib_id "Device:C") (at 212.09 68.58 0) (unit 1)
     (in_bom yes) (on_board yes)
@@
       (reference "R9") (unit 1) (value "1k5") (footprint "Resistor_SMD:R_0805_2012Metric_Pad1.20x1.40mm_HandSolder")
     )
+    (path "/9cf70606-6446-435e-8baf-5f19b839292d"
+      (reference "R10") (unit 1) (value "0R47") (footprint "Resistor_SMD:R_1206_3216Metric_Pad1.30x1.75mm_HandSolder")
+    )
     (path "/00000000-0000-0000-0000-0000606e4326"

Commit message: WIP
Parts:
- added R11: 0R47, Resistor_SMD:R_0805_2012Metric_Pad1.20x1.40mm_HandSolder, symbol Device:R
- R10: footprint Resistor_SMD:R_1206_3216Metric_Pad1.30x1.75mm_HandSolder -> Resistor_SMD:R_0805_2012Metric_Pad1.20x1.40mm_HandSolder
Connections:
- net GND: now also R11.1
- net at R10.2, U2.7 (RS): now also R11.2
Other:
- moved on the sheet: R10
Changed lines of the file:
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@@
   (junction (at 57.15 72.39) (diameter 0) (color 0 0 0 0)
   )
+  (junction (at 232.41 74.93) (diameter 0) (color 0 0 0 0)
+  )
   (junction (at 50.8 52.07) (diameter 0) (color 0 0 0 0)
   )
@@
   (junction (at 57.15 48.26) (diameter 0) (color 0 0 0 0)
   )
+  (junction (at 232.41 86.36) (diameter 0) (color 0 0 0 0)
+  )
   (junction (at 50.8 72.39) (diameter 0) (color 0 0 0 0)
   )
   (junction (at 63.5 52.07) (diameter 0) (color 0 0 0 0)
   )
-  (junction (at 229.87 83.82) (diameter 0) (color 0 0 0 0)
+  (junction (at 229.87 86.36) (diameter 0) (color 0 0 0 0)
   )
   (no_connect (at 110.49 60.96))
@@
     (stroke (width 0) (type default) (color 0 0 0 0))
   )
+  (wire (pts (xy 237.49 86.36) (xy 237.49 83.82))
+    (stroke (width 0) (type default) (color 0 0 0 0))
+  )
   (wire (pts (xy 149.86 127) (xy 152.4 127))
     (stroke (width 0) (type default) (color 0 0 0 0))
@@
     (stroke (width 0) (type default) (color 0 0 0 0))
   )
-  (wire (pts (xy 232.41 81.28) (xy 232.41 83.82))
+  (wire (pts (xy 232.41 83.82) (xy 232.41 86.36))
     (stroke (width 0) (type default) (color 0 0 0 0))
   )
@@
     (stroke (width 0) (type default) (color 0 0 0 0))
   )
-  (wire (pts (xy 232.41 83.82) (xy 229.87 83.82))
-    (stroke (width 0) (type default) (color 0 0 0 0))
-  )
-  (wire (pts (xy 229.87 73.66) (xy 229.87 83.82))
+  (wire (pts (xy 232.41 86.36) (xy 229.87 86.36))
+    (stroke (width 0) (type default) (color 0 0 0 0))
+  )
+  (wire (pts (xy 229.87 73.66) (xy 229.87 86.36))
+    (stroke (width 0) (type default) (color 0 0 0 0))
+  )
+  (wire (pts (xy 237.49 74.93) (xy 237.49 76.2))
     (stroke (width 0) (type default) (color 0 0 0 0))
   )
@@
     (stroke (width 0) (type default) (color 0 0 0 0))
   )
+  (wire (pts (xy 232.41 74.93) (xy 237.49 74.93))
+    (stroke (width 0) (type default) (color 0 0 0 0))
+  )
   (wire (pts (xy 187.96 129.54) (xy 246.38 129.54))
     (stroke (width 0) (type default) (color 0 0 0 0))
@@
     (stroke (width 0) (type default) (color 0 0 0 0))
   )
+  (wire (pts (xy 232.41 86.36) (xy 237.49 86.36))
+    (stroke (width 0) (type default) (color 0 0 0 0))
+  )
   (wire (pts (xy 50.8 48.26) (xy 57.15 48.26))
     (stroke (width 0) (type default) (color 0 0 0 0))
@@
     (stroke (width 0) (type default) (color 0 0 0 0))
   )
-  (wire (pts (xy 227.33 73.66) (xy 227.33 83.82))
-    (stroke (width 0) (type default) (color 0 0 0 0))
-  )
-  (wire (pts (xy 227.33 83.82) (xy 229.87 83.82))
-    (stroke (width 0) (type default) (color 0 0 0 0))
-  )
-  (wire (pts (xy 229.87 83.82) (xy 229.87 85.09))
+  (wire (pts (xy 227.33 73.66) (xy 227.33 86.36))
+    (stroke (width 0) (type default) (color 0 0 0 0))
+  )
+  (wire (pts (xy 227.33 86.36) (xy 229.87 86.36))
+    (stroke (width 0) (type default) (color 0 0 0 0))
+  )
+  (wire (pts (xy 229.87 86.36) (xy 229.87 87.63))
     (stroke (width 0) (type default) (color 0 0 0 0))
   )
   (wire (pts (xy 233.68 127) (xy 233.68 123.19))
+    (stroke (width 0) (type default) (color 0 0 0 0))
+  )
+  (wire (pts (xy 232.41 76.2) (xy 232.41 74.93))
+    (stroke (width 0) (type default) (color 0 0 0 0))
+  )
+  (wire (pts (xy 232.41 74.93) (xy 232.41 73.66))
     (stroke (width 0) (type default) (color 0 0 0 0))
   )
@@
     (pin "1")
   )
-  (symbol (lib_id "power:GND") (at 229.87 85.09 0) (unit 1)
-    (in_bom yes) (on_board yes)
-    (property "Reference" "#PWR023" (id 0) (at 229.87 91.44 0)
-      (effects (font (size 1.27 1.27)) hide)
-    )
-    (property "Value" "GND" (id 1) (at 229.997 89.4842 0))
-    (property "Footprint" "" (id 2) (at 229.87 85.09 0)
-      (effects (font (size 1.27 1.27)) hide)
-    )
-    (property "Datasheet" "" (id 3) (at 229.87 85.09 0)
+  (symbol (lib_id "power:GND") (at 229.87 87.63 0) (unit 1)
+    (in_bom yes) (on_board yes)
+    (property "Reference" "#PWR023" (id 0) (at 229.87 93.98 0)
+      (effects (font (size 1.27 1.27)) hide)
+    )
+    (property "Value" "GND" (id 1) (at 229.997 92.0242 0))
+    (property "Footprint" "" (id 2) (at 229.87 87.63 0)
+      (effects (font (size 1.27 1.27)) hide)
+    )
+    (property "Datasheet" "" (id 3) (at 229.87 87.63 0)
       (effects (font (size 1.27 1.27)) hide)
     )
@@
     (pin "1")
   )
+  (symbol (lib_id "Device:R") (at 237.49 80.01 180) (unit 1)
+    (in_bom yes) (on_board yes)
+    (property "Reference" "R11" (id 0) (at 240.03 83.82 90))
+    (property "Value" "0R47" (id 1) (at 240.03 78.74 90))
+    (property "Footprint" "Resistor_SMD:R_0805_2012Metric_Pad1.20x1.40mm_HandSolder" (id 2) (at 239.268 80.01 90)
+      (effects (font (size 1.27 1.27)) hide)
+    )
+    (property "Datasheet" "~" (id 3) (at 237.49 80.01 0)
+      (effects (font (size 1.27 1.27)) hide)
+    )
+    (pin "1")
+    (pin "2")
+  )
   (symbol (lib_id "power:GND") (at 212.09 72.39 0) (unit 1)
     (in_bom yes) (on_board yes)
@@
     (pin "1")
   )
-  (symbol (lib_id "Device:R") (at 232.41 77.47 180) (unit 1)
-    (in_bom yes) (on_board yes)
-    (property "Reference" "R10" (id 0) (at 237.6678 77.47 90))
-    (property "Value" "0R47" (id 1) (at 235.3564 77.47 90))
-    (property "Footprint" "Resistor_SMD:R_1206_3216Metric_Pad1.30x1.75mm_HandSolder" (id 2) (at 234.188 77.47 90)
-      (effects (font (size 1.27 1.27)) hide)
-    )
-    (property "Datasheet" "~" (id 3) (at 232.41 77.47 0)
+  (symbol (lib_id "Device:R") (at 232.41 80.01 180) (unit 1)
+    (in_bom yes) (on_board yes)
+    (property "Reference" "R10" (id 0) (at 234.95 83.82 90))
+    (property "Value" "0R47" (id 1) (at 234.95 78.74 90))
+    (property "Footprint" "Resistor_SMD:R_0805_2012Metric_Pad1.20x1.40mm_HandSolder" (id 2) (at 234.188 80.01 90)
+      (effects (font (size 1.27 1.27)) hide)
+    )
+    (property "Datasheet" "~" (id 3) (at 232.41 80.01 0)
       (effects (font (size 1.27 1.27)) hide)
     )
@@
     )
     (path "/9cf70606-6446-435e-8baf-5f19b839292d"
-      (reference "R10") (unit 1) (value "0R47") (footprint "Resistor_SMD:R_1206_3216Metric_Pad1.30x1.75mm_HandSolder")
+      (reference "R10") (unit 1) (value "0R47") (footprint "Resistor_SMD:R_0805_2012Metric_Pad1.20x1.40mm_HandSolder")
+    )
+    (path "/4f7770dd-4b94-4adc-acb1-e53a5fecd595"
+      (reference "R11") (unit 1) (value "0R47") (footprint "Resistor_SMD:R_0805_2012Metric_Pad1.20x1.40mm_HandSolder")
     )
     (path "/00000000-0000-0000-0000-0000606e4326"
