File: t100-relay/board/t100-relay.kicad_pcb (KiCad board)
At the start: 2 copper layers, 34.5 x 99.5 mm, 14 parts, among them J1 T100-IN, J2 T100-OUT, J3 Conn_01x02_Female, J4 Conn_01x02_Female, K1 RELAY_2, Q1 BC817, U1 ATSAMD09C13A-SS, X1 SWD

Commit message: WIP
Parts:
- K1: value RELAY_2 -> RELAY_1; footprint Drake:RT314_Relay -> Drake:SRD_C_Relay
- moved C1 38.4 mm to (93.0, 89.0), turned to 0 degrees
- moved D1 26.1 mm to (86.0, 93.0), turned to 180 degrees
- moved R1 20.9 mm to (86.0, 90.0), turned to 0 degrees
- moved D2 18.6 mm to (94.0, 102.0), turned to 180 degrees
- moved Q1 14.6 mm to (86.0, 102.5)
- moved J2 14.2 mm to (93.0, 85.1)
- moved JP1 13.6 mm to (90.5, 70.5)
- moved J4 11.2 mm to (96.2, 124.5)
- moved R2 8.25 mm to (86.0, 98.5)
- moved X1 6.04 mm to (100.5, 91.0)
- moved J3 4.25 mm to (86.2, 124.5)
- moved U1 3.16 mm to (93.5, 94.5)
- moved K1 2.78 mm to (84.8, 113.0)
Connections:
- K1 pad 2: Net-(D2-Pad2) -> Net-(J4-Pad2)
Routing:
- net +5V: track 19.5 -> 67.6 mm
- net +12V: track 49.2 -> 15.6 mm
- net Net-(J3-Pad1): track 0.00 -> 26.5 mm
- net /ADDR: track 0.00 -> 22.8 mm
- net Net-(J3-Pad2): track 0.00 -> 20.5 mm
- net +3V3: track 19.5 -> 31.7 mm
- net Net-(J4-Pad2): track 0.00 -> 10.9 mm
- net /RST: track 19.5 -> 30.2 mm, vias 0 -> 2
- net GND: track 39.0 -> 29.3 mm, vias 0 -> 2
- net Net-(D2-Pad2): track 0.00 -> 9.11 mm
- net /RELAY: track 0.00 -> 5.61 mm
- net /SWCLK: track 0.00 -> 5.37 mm
- net /SWDIO: track 0.00 -> 5.28 mm
- net /SDA: track 19.5 -> 24.0 mm, vias 0 -> 2
- net Net-(Q1-Pad1): track 0.00 -> 3.85 mm
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Other:
- board size 34.5 x 99.5 mm -> 20.3 x 99.5 mm
- board text added: "MAX 10A 250VAC"
- board text added: "POWER RELAY v1.0"
- board text added: "SWD"
- board text removed: "230V 16A RELAY v1.0"
- board text removed: "ADDR"

Commit message: WIP
Parts:
- moved J3 13.3 mm to (86.8, 137.8)
- moved J4 13.3 mm to (96.8, 137.8)
- moved K1 4.00 mm to (84.8, 117.0)
- moved J1 0.35 mm to (88.0, 84.9)
- moved J2 0.25 mm to (93.0, 84.9)
Routing:
- net +5V: track 67.6 -> 5.00 mm
- net GND: track 29.3 -> 0.00 mm, vias 2 -> 0
- net +3V3: track 31.7 -> 5.00 mm
- net Net-(J3-Pad1): track 26.5 -> 0.00 mm
- net /RST: track 30.2 -> 5.00 mm, vias 2 -> 0
- net /ADDR: track 22.8 -> 0.00 mm
- net Net-(J3-Pad2): track 20.5 -> 0.00 mm
- net /SDA: track 24.0 -> 5.00 mm, vias 2 -> 0
- net /IRQ: track 21.9 -> 5.00 mm
- net /SCL: track 21.0 -> 5.00 mm, vias 2 -> 0
- net Net-(J4-Pad2): track 10.9 -> 0.00 mm
- net Net-(D2-Pad2): track 9.11 -> 0.00 mm
- net /RELAY: track 5.61 -> 0.00 mm
- net /SWCLK: track 5.37 -> 0.00 mm
- net /SWDIO: track 5.28 -> 0.00 mm
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Other:
- board size 20.3 x 99.5 mm -> 20 x 100 mm

Commit message: WIP
Routing:
- net Net-(J3-Pad2): track 0.00 -> 32.5 mm
- net Net-(J4-Pad2): track 0.00 -> 20.4 mm
- net Net-(J3-Pad1): track 0.00 -> 10.0 mm
Other:
- board text added: "T100-RELAY v1.0"
- board text removed: "POWER RELAY v1.0"
Changed lines of the file:
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@@
   (gr_line (start 92 137.2) (end 92 134) (layer "F.SilkS") (width 0.12))
   (gr_line (start 102 137.2) (end 94 137.2) (layer "F.SilkS") (width 0.12))
+  (gr_line (start 83.5 52) (end 102.5 52) (layer "F.SilkS") (width 0.12))
   (gr_line (start 92 137.2) (end 84 137.2) (layer "F.SilkS") (width 0.12))
   (gr_line (start 102 137.2) (end 102 134) (layer "F.SilkS") (width 0.12))
@@
   (gr_circle (center 93 130) (end 94.75 130) (layer "Edge.Cuts") (width 0.2) (fill none))
   (gr_line (start 107.25 62.249999) (end 87.75 62.249999) (layer "F.Fab") (width 0.254))
-  (gr_text "POWER RELAY v1.0" (at 93 59.5) (layer "F.SilkS")
+  (gr_text "T100-RELAY v1.0" (at 93 51) (layer "F.SilkS")
     (effects (font (size 1 1) (thickness 0.2)))
   )
@@
   (segment (start 88 82.32) (end 93 82.32) (width 2) (layer "B.Cu") (net 8))
   (segment (start 88 74.7) (end 93 74.7) (width 2) (layer "B.Cu") (net 13))
+  (segment (start 96.79 137.75) (end 96.79 142.75) (width 2.5) (layer "B.Cu") (net 15))
+  (segment (start 86.79 142.75) (end 86.79 137.75) (width 2.5) (layer "B.Cu") (net 15))
+  (segment (start 91 125) (end 88 128) (width 2.5) (layer "B.Cu") (net 16))
+  (segment (start 91 120) (end 91 125) (width 2.5) (layer "B.Cu") (net 16))
+  (segment (start 90.6 137.75) (end 90.6 142.75) (width 2.5) (layer "B.Cu") (net 16))
+  (segment (start 84.85 117) (end 88 117) (width 2.5) (layer "B.Cu") (net 16))
+  (segment (start 88 132) (end 90.6 134.6) (width 2.5) (layer "B.Cu") (net 16))
+  (segment (start 90.6 134.6) (end 90.6 137.75) (width 2.5) (layer "B.Cu") (net 16))
+  (segment (start 88 117) (end 91 120) (width 2.5) (layer "B.Cu") (net 16))
+  (segment (start 88 128) (end 88 132) (width 2.5) (layer "B.Cu") (net 16))
+  (segment (start 100.6 137.75) (end 100.6 142.75) (width 2.5) (layer "B.Cu") (net 17))
+  (segment (start 99.05 123) (end 100.6 124.55) (width 2.5) (layer "B.Cu") (net 17))
+  (segment (start 100.6 124.55) (end 100.6 137.75) (width 2.5) (layer "B.Cu") (net 17))
   (zone (net 1) (net_name "GND") (layer "B.Cu") (hatch edge 0.508)
     (connect_pads (clearance 0.508))

Commit message: WIP
Parts:
- moved JP1 19.6 mm to (86.8, 89.8), turned to 180 degrees
- moved D2 3.16 mm to (97.0, 103.0)
- moved Q1 3.04 mm to (89.0, 103.0)
- moved R1 2.80 mm to (85.5, 92.8)
- moved D1 2.30 mm to (85.5, 95.2)
- moved U1 1.68 mm to (92.0, 95.2)
- moved C1 1.44 mm to (91.8, 89.8)
- moved R2 0.90 mm to (85.5, 97.8), turned to 180 degrees
- moved X1 0.75 mm to (100.5, 91.8)
Routing:
- net +5V: track 5.00 -> 68.5 mm
- net /RST: track 5.00 -> 33.4 mm
- net /SDA: track 5.00 -> 32.9 mm
- net +3V3: track 5.00 -> 29.1 mm
- net /SCL: track 5.00 -> 26.1 mm
- net /IRQ: track 5.00 -> 26.0 mm
- net Net-(D2-Pad2): track 0.00 -> 16.9 mm
- net Net-(J3-Pad1): track 10.0 -> 23.9 mm
- net GND: track 0.00 -> 13.2 mm, vias 0 -> 6
- net /SWDIO: track 0.00 -> 7.97 mm, vias 0 -> 1
- net Net-(Q1-Pad1): track 0.00 -> 6.22 mm
- net /SWCLK: track 0.00 -> 6.11 mm
- net /ADDR: track 0.00 -> 4.75 mm
- net Net-(D1-Pad2): track 0.00 -> 2.51 mm
- net /RELAY: track 0.00 -> 1.70 mm
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
Commit message: WIP
Routing:
- net GND: track 13.2 -> 18.2 mm
- net +3V3: track 29.1 -> 28.1 mm
Changed lines of the file:
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@@
     (effects (font (size 1 1) (thickness 0.15)))
   )
-  (gr_text "B" (at 88.25 87.5) (layer "F.SilkS")
+  (gr_text "B" (at 85 87.5) (layer "F.SilkS")
     (effects (font (size 1 1) (thickness 0.15)))
   )
@@
     (effects (font (size 1 1) (thickness 0.15)))
   )
-  (gr_text "A" (at 85.25 87.5) (layer "F.SilkS")
+  (gr_text "A" (at 88.5 87.5) (layer "F.SilkS")
     (effects (font (size 1 1) (thickness 0.15)))
   )
@@
   (segment (start 92 92.775) (end 92 90.55625) (width 0.4) (layer "F.Cu") (net 1))
   (segment (start 85.625 102.375) (end 84.875 101.625) (width 0.6) (layer "F.Cu") (net 1))
+  (segment (start 88 62) (end 93 62) (width 2) (layer "F.Cu") (net 1))
   (segment (start 84.75 89.76875) (end 84.76875 89.75) (width 0.4) (layer "F.Cu") (net 1))
   (segment (start 92 90.55625) (end 92.80625 89.75) (width 0.4) (layer "F.Cu") (net 1))
@@
   (via (at 84.875 101.625) (size 0.8) (drill 0.4) (layers "F.Cu" "B.Cu") (net 1))
   (via (at 84.75 91.25) (size 0.8) (drill 0.4) (layers "F.Cu" "B.Cu") (net 1))
+  (segment (start 89.75 87.5) (end 89.75 72) (width 0.4) (layer "F.Cu") (net 2))
+  (segment (start 88.76875 89.75) (end 90.73125 89.75) (width 0.4) (layer "F.Cu") (net 2))
+  (segment (start 90.73125 89.75) (end 90.73125 88.48125) (width 0.4) (layer "F.Cu") (net 2))
+  (segment (start 90.73125 89.75) (end 90.73125 92.77375) (width 0.4) (layer "F.Cu") (net 2))
   (segment (start 90.73125 88.48125) (end 89.75 87.5) (width 0.4) (layer "F.Cu") (net 2))
-  (segment (start 88.76875 89.75) (end 90.73125 89.75) (width 0.4) (layer "F.Cu") (net 2))
-  (segment (start 89.75 73.25) (end 88.66 72.16) (width 0.4) (layer "F.Cu") (net 2))
-  (segment (start 89.75 87.5) (end 89.75 73.25) (width 0.4) (layer "F.Cu") (net 2))
-  (segment (start 90.73125 89.75) (end 90.73125 92.77375) (width 0.4) (layer "F.Cu") (net 2))
-  (segment (start 90.73125 89.75) (end 90.73125 88.48125) (width 0.4) (layer "F.Cu") (net 2))
   (segment (start 90.73125 92.77375) (end 90.73 92.775) (width 0.4) (layer "F.Cu") (net 2))
-  (segment (start 88.66 72.16) (end 88 72.16) (width 0.4) (layer "F.Cu") (net 2))
-  (segment (start 88 72.16) (end 93 72.16) (width 2) (layer "B.Cu") (net 2))
-  (segment (start 88 64.54) (end 93 64.54) (width 2) (layer "B.Cu") (net 3))
-  (segment (start 88 67.08) (end 93 67.08) (width 2) (layer "B.Cu") (net 3))
-  (segment (start 93 64.54) (end 93 67.08) (width 2) (layer "B.Cu") (net 3))
-  (segment (start 88 64.54) (end 88 67.08) (width 2) (layer "B.Cu") (net 3))
+  (segment (start 93 72.16) (end 88 72.16) (width 2) (layer "F.Cu") (net 2))
+  (segment (start 88 64.54) (end 88 67.08) (width 2) (layer "F.Cu") (net 3))
+  (segment (start 88 67.08) (end 93 67.08) (width 2) (layer "F.Cu") (net 3))
+  (segment (start 93 64.54) (end 88 64.54) (width 2) (layer "F.Cu") (net 3))
+  (segment (start 93 67.08) (end 93 64.54) (width 2) (layer "F.Cu") (net 3))
   (segment (start 84.5 92.75) (end 84.5 95.225) (width 0.4) (layer "F.Cu") (net 4))
   (segment (start 84.5 95.225) (end 84.475 95.25) (width 0.4) (layer "F.Cu") (net 4))
   (segment (start 93.12 69.62) (end 93 69.62) (width 0.6) (layer "F.Cu") (net 5))
+  (segment (start 93 69.62) (end 88 69.62) (width 2) (layer "F.Cu") (net 5))
   (segment (start 102 78.5) (end 93.12 69.62) (width 0.6) (layer "F.Cu") (net 5))
   (segment (start 93 109.7) (end 99.7 103) (width 0.6) (layer "F.Cu") (net 5))
@@
   (segment (start 99.7 103) (end 102 100.7) (width 0.6) (layer "F.Cu") (net 5))
   (segment (start 102 100.7) (end 102 78.5) (width 0.6) (layer "F.Cu") (net 5))
-  (segment (start 88 69.62) (end 93 69.62) (width 2) (layer "B.Cu") (net 5))
   (segment (start 95.25 88.75) (end 94.5 88) (width 0.4) (layer "F.Cu") (net 6))
   (segment (start 90.5 87) (end 90.5 79) (width 0.4) (layer "F.Cu") (net 6))
@@
     (polygon
       (pts
-        (xy 103.5 103.5)
-        (xy 82.5 103.5)
-        (xy 82.5 50)
-        (xy 103.5 50)
+        (xy 103 103.5)
+        (xy 83 103.5)
+        (xy 83 50)
+        (xy 103 50)
       )
     )
+  )
+  (zone (net 0) (net_name "") (layer "B.Mask") (hatch edge 0.508)
+    (connect_pads (clearance 0))
+    (min_thickness 0.254) (filled_areas_thickness no)
+    (fill yes (thermal_gap 0.508) (thermal_bridge_width 0.508))
+    (polygon
+      (pts
+        (xy 89 115)
+        (xy 95 121)
+        (xy 100 121)
+        (xy 103 124)
+        (xy 103 143)
+        (xy 98 148)
+        (xy 87 148)
+        (xy 83 144)
+        (xy 83 115)
+      )
+    )
