File: t100-psu/board/t100-psu.kicad_sch (KiCad schematic)
At the start: 23 parts, among them J1 Conn_01x02_Female, J2 T100-IN, J3 T100-OUT, U1 FR8205, U2 FR8205

Commit message: WIP
Parts:
- renumbered DW1 to D1
Changed lines of the file:
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@@
 (kicad_sch (version 20210621) (generator eeschema)
   (paper "A4")
-  (junction (at 158.75 104.14) (diameter 0) (color 0 0 0 0))
-  (junction (at 158.75 76.2) (diameter 0) (color 0 0 0 0))
+  (junction (at 135.89 124.46) (diameter 0) (color 0 0 0 0))
   (junction (at 119.38 104.14) (diameter 0) (color 0 0 0 0))
-  (junction (at 149.86 55.88) (diameter 0) (color 0 0 0 0))
-  (junction (at 158.75 114.3) (diameter 0) (color 0 0 0 0))
-  (junction (at 158.75 124.46) (diameter 0) (color 0 0 0 0))
-  (junction (at 168.91 55.88) (diameter 0) (color 0 0 0 0))
-  (junction (at 119.38 55.88) (diameter 0) (color 0 0 0 0))
-  (junction (at 119.38 124.46) (diameter 0) (color 0 0 0 0))
-  (junction (at 111.76 104.14) (diameter 0) (color 0 0 0 0))
-  (junction (at 229.87 121.92) (diameter 0) (color 0 0 0 0))
-  (junction (at 135.89 124.46) (diameter 0) (color 0 0 0 0))
   (junction (at 111.76 55.88) (diameter 0) (color 0 0 0 0))
-  (junction (at 168.91 104.14) (diameter 0) (color 0 0 0 0))
   (junction (at 135.89 76.2) (diameter 0) (color 0 0 0 0))
   (junction (at 119.38 76.2) (diameter 0) (color 0 0 0 0))
+  (junction (at 111.76 104.14) (diameter 0) (color 0 0 0 0))
+  (junction (at 168.91 104.14) (diameter 0) (color 0 0 0 0))
+  (junction (at 158.75 76.2) (diameter 0) (color 0 0 0 0))
+  (junction (at 158.75 124.46) (diameter 0) (color 0 0 0 0))
+  (junction (at 119.38 55.88) (diameter 0) (color 0 0 0 0))
+  (junction (at 229.87 82.55) (diameter 0) (color 0 0 0 0))
+  (junction (at 158.75 114.3) (diameter 0) (color 0 0 0 0))
+  (junction (at 158.75 66.04) (diameter 0) (color 0 0 0 0))
+  (junction (at 168.91 55.88) (diameter 0) (color 0 0 0 0))
+  (junction (at 119.38 124.46) (diameter 0) (color 0 0 0 0))
+  (junction (at 229.87 121.92) (diameter 0) (color 0 0 0 0))
+  (junction (at 149.86 55.88) (diameter 0) (color 0 0 0 0))
+  (junction (at 158.75 104.14) (diameter 0) (color 0 0 0 0))
+  (junction (at 158.75 55.88) (diameter 0) (color 0 0 0 0))
   (junction (at 149.86 104.14) (diameter 0) (color 0 0 0 0))
-  (junction (at 158.75 66.04) (diameter 0) (color 0 0 0 0))
-  (junction (at 229.87 82.55) (diameter 0) (color 0 0 0 0))
-  (junction (at 158.75 55.88) (diameter 0) (color 0 0 0 0))
   (wire (pts (xy 149.86 95.25) (xy 148.59 95.25))
     (stroke (width 0) (type default) (color 0 0 0 0))
@@
   (symbol (lib_id "Device:LED") (at 52.07 116.84 180) (unit 1)
     (in_bom yes) (on_board yes)
-    (property "Reference" "DW1" (id 0) (at 52.2478 110.363 0))
+    (property "Reference" "D1" (id 0) (at 52.2478 110.363 0))
     (property "Value" "WHITE" (id 1) (at 52.2478 112.6744 0))
     (property "Footprint" "LED_SMD:LED_0805_2012Metric_Pad1.15x1.40mm_HandSolder" (id 2) (at 52.07 116.84 0)
@@
     )
     (path "/00000000-0000-0000-0000-000060209071"
-      (reference "DW1") (unit 1) (value "WHITE") (footprint "LED_SMD:LED_0805_2012Metric_Pad1.15x1.40mm_HandSolder")
+      (reference "D1") (unit 1) (value "WHITE") (footprint "LED_SMD:LED_0805_2012Metric_Pad1.15x1.40mm_HandSolder")
     )
     (path "/00000000-0000-0000-0000-00006011c99d"
