File: t100-psu/board/t100-psu.kicad_pcb (KiCad board)
At the start: 2 copper layers, 20 x 100 mm, 23 parts, among them J1 Conn_01x02_Female, J2 T100-IN, J3 T100-OUT, U1 FR8205, U2 FR8205

Commit message: WIP
Parts:
- removed DW1: WHITE, LED_SMD:LED_0805_2012Metric_Pad1.15x1.40mm_HandSolder
- added D1: WHITE, LED_SMD:LED_0805_2012Metric_Pad1.15x1.40mm_HandSolder, F.Cu at (128.0, 60.0)
- moved R1 30.3 mm to (128.0, 63.0), turned to 180 degrees
- moved J1 7.75 mm to (118.8, 142.5)
- moved R2 6.32 mm to (125.0, 121.0), turned to 0 degrees
- moved R3 6.32 mm to (115.0, 121.0), turned to 0 degrees
- moved C3 5.59 mm to (118.0, 117.5), turned to 180 degrees
- moved C4 5.59 mm to (128.0, 117.5), turned to 180 degrees
- moved U1 4.12 mm to (123.0, 118.0), turned to 0 degrees
- moved U2 4.12 mm to (113.0, 118.0), turned to 0 degrees
- moved C5 4.00 mm to (123.0, 115.0), turned to 0 degrees
- moved C6 4.00 mm to (113.0, 115.0), turned to 0 degrees
- moved J2 2.50 mm to (112.5, 89.9)
- moved J3 2.50 mm to (122.5, 89.9)
Routing:
- net +12V: track 0.00 -> 160.8 mm
- net +3V3: track 0.00 -> 68.7 mm
- net +5V: track 0.00 -> 59.4 mm
- net GND: track 0.00 -> 43.5 mm, vias 0 -> 17
- net Net-(R6-Pad1): track 0.00 -> 22.4 mm, vias 0 -> 2
- net Net-(R4-Pad1): track 0.00 -> 21.4 mm, vias 0 -> 2
- net /SDA: track 0.00 -> 10.0 mm
- net /SCL: track 0.00 -> 10.0 mm
- net /RST: track 0.00 -> 10.0 mm
- net /IRQ: track 0.00 -> 10.0 mm
- net Net-(C5-Pad2): track 0.00 -> 7.24 mm
- net Net-(C6-Pad2): track 0.00 -> 7.16 mm
- net Net-(D1-Pad1): track 0.00 -> 3.05 mm
- net Net-(C5-Pad1): track 0.00 -> 1.50 mm
- net Net-(C6-Pad1): track 0.00 -> 1.45 mm
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- added copper zone on B.Cu, net GND
Other:
- board size 20 x 100 mm -> 25 x 100 mm
- board text added: "12V"
- board text added: "3V3"
- board text added: "5V"
- board text added: "GND"
- board text added: "IRQ"
- board text added: "RST"
- board text added: "SCL"
- board text added: "SDA"
- board text added: "T100-PSU v1.0"

Commit message: WIP
Changed lines of the file:
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@@
     (property "Sheetname" "")
     (attr smd)
-    (fp_text reference "U1" (at -3.000001 2.75 90) (layer "F.SilkS")
+    (fp_text reference "U1" (at -0.000001 2.75 90) (layer "F.SilkS")
       (effects (font (size 1 1) (thickness 0.15)))
     )
@@
     (fp_line (start 0.8 1.45) (end -0.8 1.45) (layer "F.Fab") (width 0.1))
     (pad "1" smd roundrect locked (at -1.1375 -0.95) (size 1.325 0.6) (layers "F.Cu" "F.Paste" "F.Mask") (roundrect_rratio 0.25)
-      (net 3 "Net-(C5-Pad1)") (pinfunction "BST") (pintype "bidirectional"))
+      (net 3 "Net-(C5-Pad1)") (pinfunction "BST"))
     (pad "2" smd roundrect locked (at -1.1375 0) (size 1.325 0.6) (layers "F.Cu" "F.Paste" "F.Mask") (roundrect_rratio 0.25)
-      (net 2 "GND") (pinfunction "GND") (pintype "power_in"))
+      (net 2 "GND") (pinfunction "GND"))
     (pad "3" smd roundrect locked (at -1.1375 0.95) (size 1.325 0.6) (layers "F.Cu" "F.Paste" "F.Mask") (roundrect_rratio 0.25)
-      (net 16 "Net-(R4-Pad1)") (pinfunction "FB") (pintype "input"))
+      (net 16 "Net-(R4-Pad1)") (pinfunction "FB"))
     (pad "4" smd roundrect locked (at 1.1375 0.95) (size 1.325 0.6) (layers "F.Cu" "F.Paste" "F.Mask") (roundrect_rratio 0.25)
-      (net 14 "Net-(R2-Pad1)") (pinfunction "SHDN") (pintype "input"))
+      (net 14 "Net-(R2-Pad1)") (pinfunction "SHDN"))
     (pad "5" smd roundrect locked (at 1.1375 0) (size 1.325 0.6) (layers "F.Cu" "F.Paste" "F.Mask") (roundrect_rratio 0.25)
-      (net 1 "+12V") (pinfunction "VIN") (pintype "power_in"))
+      (net 1 "+12V") (pinfunction "VIN"))
     (pad "6" smd roundrect locked (at 1.1375 -0.95) (size 1.325 0.6) (layers "F.Cu" "F.Paste" "F.Mask") (roundrect_rratio 0.25)
-      (net 4 "Net-(C5-Pad2)") (pinfunction "LX") (pintype "power_out"))
+      (net 4 "Net-(C5-Pad2)") (pinfunction "LX"))
     (model "${KICAD6_3DMODEL_DIR}/Package_TO_SOT_SMD.3dshapes/SOT-23-6.wrl"
       (offset (xyz 0 0 0))
@@
     (property "Sheetname" "")
     (attr smd)
-    (fp_text reference "U2" (at -3.000001 2.75 90) (layer "F.SilkS")
+    (fp_text reference "U2" (at -0.000001 2.75 90) (layer "F.SilkS")
       (effects (font (size 1 1) (thickness 0.15)))
     )
@@
     (property "Sheetname" "")
     (attr smd)
-    (fp_text reference "C5" (at 2.749999 0) (layer "F.SilkS")
+    (fp_text reference "C5" (at 2.749999 -0.5) (layer "F.SilkS")
       (effects (font (size 1 1) (thickness 0.15)))
     )
@@
     (property "Sheetname" "")
     (attr smd)
-    (fp_text reference "C6" (at 2.999999 0) (layer "F.SilkS")
-      (effects (font (size 1 1) (thickness 0.15)))
-    )
+    (fp_text reference "C6" (at 2.999999 -0.5) (layer "F.SilkS")
+      (effects (font (size 1 1) (thickness 0.15)))
+    )

Commit message: WIP
Other:
- board text added: "T100-PSU v2.0"
- board text removed: "T100-PSU v1.0"
Changed lines of the file:
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@@
     (effects (font (size 1 1) (thickness 0.15)))
   )
-  (gr_text "T100-PSU v1.0" (at 120 56) (layer "F.SilkS")
+  (gr_text "T100-PSU v2.0" (at 120 56) (layer "F.SilkS")
     (effects (font (size 1 1) (thickness 0.15)))
   )

Commit message: WIP
Routing:
- net GND: track 43.5 -> 53.5 mm
- net +12V: track 160.8 -> 170.8 mm
- net +3V3: track 68.7 -> 75.5 mm
Changed lines of the file:
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@@
   (segment (start 121 126) (end 120 126) (width 2) (layer "F.Cu") (net 1))
   (segment (start 122.600001 147.5) (end 122.600001 142.5) (width 2) (layer "F.Cu") (net 1))
+  (segment (start 122.5 72.08) (end 112.5 72.08) (width 2) (layer "F.Cu") (net 1))
   (segment (start 123.25 125.25) (end 123.25 127.25) (width 2) (layer "F.Cu") (net 1))
   (segment (start 126 139.100001) (end 122.600001 142.5) (width 2) (layer "F.Cu") (net 1))
   (segment (start 122 126) (end 123.25 127.25) (width 2) (layer "F.Cu") (net 1))
+  (segment (start 122.5 69.54) (end 122.5 72.08) (width 2) (layer "F.Cu") (net 1))
   (segment (start 126 130) (end 126 139.100001) (width 2) (layer "F.Cu") (net 1))
+  (segment (start 112.5 72.08) (end 112.5 69.54) (width 2) (layer "F.Cu") (net 1))
   (segment (start 116 118) (end 114.137501 118) (width 0.6) (layer "F.Cu") (net 1))
   (segment (start 116.5 117.5) (end 116.5 124.699999) (width 2) (layer "F.Cu") (net 1))
+  (segment (start 112.5 69.54) (end 122.5 69.54) (width 2) (layer "F.Cu") (net 1))
   (segment (start 122.200001 126) (end 121 126) (width 2) (layer "F.Cu") (net 1))
-  (segment (start 122.5 69.54) (end 112.5 69.54) (width 2) (layer "B.Cu") (net 1))
   (segment (start 127.08 72.08) (end 112.5 72.08) (width 2) (layer "B.Cu") (net 1))
   (segment (start 131 76) (end 127.08 72.08) (width 2) (layer "B.Cu") (net 1))
-  (segment (start 122.5 69.54) (end 122.5 72.08) (width 2) (layer "B.Cu") (net 1))
   (segment (start 122.600001 142.5) (end 122.600001 142.399999) (width 2) (layer "B.Cu") (net 1))
-  (segment (start 112.5 69.54) (end 112.5 72.08) (width 2) (layer "B.Cu") (net 1))
   (segment (start 131 134) (end 131 76) (width 2) (layer "B.Cu") (net 1))
   (segment (start 122.600001 142.399999) (end 131 134) (width 2) (layer "B.Cu") (net 1))
@@
   (segment (start 121 118) (end 120 117) (width 0.6) (layer "F.Cu") (net 2))
   (segment (start 118.790001 147.5) (end 118.790001 142.5) (width 2) (layer "F.Cu") (net 2))
+  (segment (start 112.5 67) (end 122.5 67) (width 2) (layer "F.Cu") (net 2))
   (segment (start 110 118) (end 110 117) (width 0.4) (layer "F.Cu") (net 2))
   (segment (start 126.5 63) (end 122.5 67) (width 0.6) (layer "F.Cu") (net 2))
@@
   (segment (start 130.5 98) (end 131 97.5) (width 2) (layer "F.Cu") (net 7))
   (segment (start 127.12 74.62) (end 122.5 74.62) (width 2) (layer "F.Cu") (net 7))
+  (segment (start 122.5 74.62) (end 112.5 74.62) (width 2) (layer "F.Cu") (net 7))
   (segment (start 131 105.5) (end 131 104) (width 2) (layer "F.Cu") (net 7))
   (segment (start 127.775001 108.724999) (end 131 105.5) (width 2) (layer "F.Cu") (net 7))
@@
   (segment (start 131 97.5) (end 131 78.5) (width 2) (layer "F.Cu") (net 7))
   (segment (start 131 104) (end 131 97.5) (width 2) (layer "F.Cu") (net 7))
-  (segment (start 122.5 74.62) (end 112.5 74.62) (width 2) (layer "B.Cu") (net 7))
-  (segment (start 119 77) (end 120.22896 78.22896) (width 0.6) (layer "F.Cu") (net 8))
-  (segment (start 122.5 77.16) (end 121.297919 77.16) (width 2) (layer "F.Cu") (net 8))
-  (segment (start 119 67) (end 119 77) (width 0.6) (layer "F.Cu") (net 8))
+  (segment (start 110 66.5) (end 110 75.5) (width 0.6) (layer "F.Cu") (net 8))
   (segment (start 118.5 98.699999) (end 118.5 109.275001) (width 2) (layer "F.Cu") (net 8))
-  (segment (start 117.800001 80.657918) (end 117.800001 98) (width 2) (layer "F.Cu") (net 8))
+  (segment (start 122.5 77.16) (end 118.34 77.16) (width 2) (layer "F.Cu") (net 8))
   (segment (start 117.800001 98) (end 118.5 98.699999) (width 2) (layer "F.Cu") (net 8))
-  (segment (start 120.22896 78.22896) (end 117.800001 80.657918) (width 2) (layer "F.Cu") (net 8))
-  (segment (start 126 60) (end 119 67) (width 0.6) (layer "F.Cu") (net 8))
+  (segment (start 111.66 77.16) (end 112.5 77.16) (width 0.6) (layer "F.Cu") (net 8))
   (segment (start 118.5 109.275001) (end 117.775001 110) (width 2) (layer "F.Cu") (net 8))
-  (segment (start 126.975 60) (end 126 60) (width 0.6) (layer "F.Cu") (net 8))
-  (segment (start 121.297919 77.16) (end 120.22896 78.22896) (width 2) (layer "F.Cu") (net 8))
-  (segment (start 112.5 77.16) (end 122.5 77.16) (width 2) (layer "B.Cu") (net 8))
+  (segment (start 126.975 60) (end 126.975 60.025) (width 0.6) (layer "F.Cu") (net 8))
+  (segment (start 126.975 60.025) (end 122 65) (width 0.6) (layer "F.Cu") (net 8))
+  (segment (start 118.34 77.16) (end 112.5 77.16) (width 2) (layer "F.Cu") (net 8))
+  (segment (start 117.800001 77.699999) (end 118.34 77.16) (width 2) (layer "F.Cu") (net 8))
+  (segment (start 117.800001 98) (end 117.800001 77.699999) (width 2) (layer "F.Cu") (net 8))
+  (segment (start 110 75.5) (end 111.66 77.16) (width 0.6) (layer "F.Cu") (net 8))
+  (segment (start 111.5 65) (end 110 66.5) (width 0.6) (layer "F.Cu") (net 8))
+  (segment (start 122 65) (end 111.5 65) (width 0.6) (layer "F.Cu") (net 8))
   (segment (start 129.025 60) (end 129.025 62.8875) (width 0.6) (layer "F.Cu") (net 9))
   (segment (start 129.025 62.8875) (end 128.9125 63) (width 0.6) (layer "F.Cu") (net 9))
