File: t100-raspi-zero2w/board/t100-raspi-zero2w.kicad_pcb (KiCad board)
At the start: 2 copper layers, 49.5 x 99.5 mm, 31 parts, among them J1 USB_B_Micro, J2 UART, J3 Raspberry_Pi_2_3, J4 12V, J5 T100-OUT, U1 CH330N, U2 FR8205, U3 FR8205

Commit message: WIP
Parts:
- C1, C2: footprint Capacitor_SMD:C_0805_2012Metric_Pad1.15x1.40mm_HandSolder -> Capacitor_SMD:C_0805_2012Metric_Pad1.18x1.45mm_HandSolder
- J3: footprint Drake:Raspberry-PI-3-B-vertical -> Drake:Raspberry-Pi-Zero-2-W-horizontal-2-holes
- J4: footprint Drake:DG301-5.0-02 -> Drake:DG235-3.81-02P
- moved R6 161.6 mm to (269.0, 44.9)
- moved R3 160.2 mm to (264.4, 36.9)
- moved R10 159.4 mm to (261.3, 25.4)
- moved R5 158.9 mm to (265.8, 57.5)
- moved R4 158.5 mm to (261.5, 29.1)
- moved C11 148.6 mm to (256.0, 103.6)
- moved C3 148.6 mm to (263.0, 84.0)
- moved C5 148.6 mm to (263.0, 89.0)
- moved C7 148.6 mm to (263.0, 97.0)
- moved C9 148.6 mm to (263.0, 110.0)
- moved L1 148.6 mm to (263.0, 102.0)
- moved R1 148.6 mm to (259.0, 93.0)
- moved R7 148.6 mm to (269.0, 95.1)
- moved R8 148.6 mm to (269.0, 91.1)
- moved U2 148.6 mm to (263.0, 93.0)
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Routing:
- net +12V: track 137.4 -> 0.00 mm, vias 6 -> 0
- net GND: track 88.0 -> 0.00 mm, vias 27 -> 0
- net +3V3: track 83.2 -> 0.00 mm
- net /MY_TXD: track 80.5 -> 0.00 mm, vias 2 -> 0
- net /MY_RXD: track 76.3 -> 0.00 mm
- net +5V: track 61.7 -> 0.00 mm
- net /RST: track 51.8 -> 0.00 mm, vias 1 -> 0
- net /IRQ: track 41.5 -> 0.00 mm, vias 2 -> 0
- net Net-(R10-Pad2): track 34.9 -> 0.00 mm, vias 3 -> 0
- net Net-(C1-Pad1): track 29.7 -> 0.00 mm, vias 2 -> 0
- net Net-(R2-Pad1): track 25.2 -> 0.00 mm, vias 2 -> 0
- net /SDA: track 22.0 -> 0.00 mm
- net /SCL: track 21.9 -> 0.00 mm
- net Net-(J1-Pad2): track 11.0 -> 0.00 mm
- net Net-(R7-Pad1): track 10.7 -> 0.00 mm, vias 2 -> 0
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- removed copper zone on B.Cu, net GND
Other:
- board size 49.5 x 99.5 mm -> 30 x 100 mm
- board text added: "T100-RASPI ZERO v1.1"
- board text removed: "GND"
- board text removed: "T100-RASPI v1.1"

Commit message: WIP
Parts:
- removed C10, C3, C4, C9: 100u/12V, Capacitor_SMD:CP_Elec_6.3x5.4
- removed C11, C5, C6, C7, C8: 100n, Capacitor_SMD:C_0805_2012Metric
- removed L1, L2: 6.8uH, Drake:CKCS6028
- removed R1, R2: 100k, Resistor_SMD:R_0805_2012Metric
- removed R10: 4.22k 1%, Resistor_SMD:R_0805_2012Metric
- removed R3, R4, R5, R6: 1K5, Resistor_SMD:R_0805_2012Metric
- removed R7: 30k 1%, Resistor_SMD:R_0805_2012Metric
- removed R8: 6.65k 1%, Resistor_SMD:R_0805_2012Metric
- removed R9: 30.9k 1%, Resistor_SMD:R_0805_2012Metric
- removed U2, U3: FR8205, Package_TO_SOT_SMD:SOT-23-6
- J3: value Raspberry_Pi_2_3 -> Raspberry_Pi_Zero_2_W; footprint Drake:Raspberry-Pi-Zero-2-W-horizontal-2-holes -> Drake:Raspberry-Pi-Zero-2-W-horizontal-4-holes
- J4: value 12V -> T100-IN; footprint Drake:DG235-3.81-02P -> Connector_PinHeader_2.54mm:PinHeader_1x10_P2.54mm_Horizontal
- moved J4 19.3 mm to (115.0, 79.9), turned to 180 degrees
- moved J5 10.4 mm to (130.0, 79.9)
- moved J3 10.00 mm to (135.2, 88.4)
Connections:
- J4 pad 2: +12V -> /SCL
Other:
- outline, holes or cut-outs redrawn
- board text removed: "+12V"

Commit message: WIP
Parts:
- J2: footprint Connector_PinHeader_2.54mm:PinHeader_1x03_P2.54mm_Vertical -> Connector_PinHeader_2.54mm:PinHeader_1x03_P2.54mm_Horizontal
- moved J2 153.6 mm to (120.0, 80.0), turned to 90 degrees
- moved C2 134.2 mm to (121.0, 132.0)
- moved C1 127.8 mm to (130.0, 132.0)
- moved J1 125.2 mm to (125.0, 143.0)
- moved U1 125.2 mm to (125.5, 133.5)

Commit message: WIP
Routing:
- net /RST: track 0.00 -> 85.0 mm
- net /MY_TXD: track 0.00 -> 83.8 mm, vias 0 -> 2
- net /IRQ: track 0.00 -> 77.0 mm
- net /MY_RXD: track 0.00 -> 63.8 mm, vias 0 -> 2
- net +5V: track 0.00 -> 49.1 mm
- net /SCL: track 0.00 -> 36.2 mm
- net +12V: track 0.00 -> 35.1 mm
- net /SDA: track 0.00 -> 34.1 mm
- net GND: track 0.00 -> 23.7 mm, vias 0 -> 7
- net Net-(C1-Pad1): track 0.00 -> 17.4 mm
- net +3V3: track 0.00 -> 15.0 mm
- net Net-(J1-Pad2): track 0.00 -> 9.64 mm
- net Net-(J1-Pad3): track 0.00 -> 4.61 mm
- net Net-(C2-Pad1): track 0.00 -> 2.62 mm
- added copper zone on B.Cu, net GND
Other:
- board text added: "PULLUPs for I2C,IRQ,RST as in USB"

Commit message: WIP
Parts:
- added C3: 100n, Capacitor_SMD:C_0805_2012Metric, F.Cu at (124.9, 67.2)
- added D1: RED, LED_SMD:LED_0805_2012Metric_Pad1.15x1.40mm_HandSolder, F.Cu at (125.0, 56.0)
- added R1: 1K5, Resistor_SMD:R_0805_2012Metric, F.Cu at (124.9, 77.3)
- added R2: 1K5, Resistor_SMD:R_0805_2012Metric, F.Cu at (124.9, 74.8)
- added R3: 1K5, Resistor_SMD:R_0805_2012Metric, F.Cu at (124.9, 72.2)
- added R4: 1K5, Resistor_SMD:R_0805_2012Metric, F.Cu at (124.9, 69.7)
- added R5: 270R, Resistor_SMD:R_0805_2012Metric, F.Cu at (120.0, 56.0)
- moved J2 36.6 mm to (121.4, 116.5), turned to 180 degrees
Routing:
- net +3V3: track 15.0 -> 49.8 mm
- net /MY_TXD: track 83.8 -> 52.8 mm, vias 2 -> 1
- net /IRQ: track 77.0 -> 106.4 mm
- net GND: track 23.7 -> 36.4 mm
- net /MY_RXD: track 63.8 -> 55.7 mm, vias 2 -> 1
- net /SCL: track 36.2 -> 42.9 mm, vias 0 -> 1
- net /SDA: track 34.1 -> 40.2 mm, vias 0 -> 1
- net /RST: track 85.0 -> 80.7 mm
- net Net-(D1-Pad1): track 0.00 -> 3.06 mm
Other:
- board text added: "GND"
- board text added: "IRQ"
- board text removed: "G"
- board text removed: "PULLUPs for I2C,IRQ,RST as in USB"
- board text removed: "UART"

Commit message: WIP
Other:
- board text added: "T100-RASPI ZERO v2.0"
- board text removed: "T100-RASPI ZERO v1.1"
Changed lines of the file:
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@@
     (effects (font (size 1 1) (thickness 0.15)) (justify left))
   )
-  (gr_text "T100-RASPI ZERO v1.1" (at 125 45.999999) (layer "F.SilkS")
+  (gr_text "T100-RASPI ZERO v2.0" (at 125 45.999999) (layer "F.SilkS")
     (effects (font (size 1 1) (thickness 0.15)))
   )
@@
   (segment (start 121 133.037499) (end 121 134.999999) (width 0.4) (layer "F.Cu") (net 1))
   (segment (start 126.30048 139.999999) (end 126.30048 140.256799) (width 0.4) (layer "F.Cu") (net 1))
+  (segment (start 130 133.037499) (end 130 134.999999) (width 0.4) (layer "F.Cu") (net 1))
   (segment (start 128 137.999999) (end 129 137.999999) (width 0.4) (layer "F.Cu") (net 1))
   (segment (start 126.30048 139.999999) (end 126.30048 137.699519) (width 0.4) (layer "F.Cu") (net 1))
   (segment (start 123.970001 63.029999) (end 130.000001 56.999999) (width 0.4) (layer "F.Cu") (net 1))
-  (segment (start 130 133.037499) (end 130 134.999999) (width 0.4) (layer "F.Cu") (net 1))
   (segment (start 121.0503 142.999999) (end 128.9497 142.999999) (width 0.4) (layer "F.Cu") (net 1))
   (segment (start 123.970001 67.159999) (end 123.970001 63.029999) (width 0.4) (layer "F.Cu") (net 1))

Commit message: WIP
Parts:
- moved C3 19.3 mm to (129.0, 86.0)
- moved D1 12.2 mm to (115.0, 49.0)
- moved R5 6.40 mm to (115.0, 52.0), turned to 180 degrees
Routing:
- net GND: track 36.4 -> 39.8 mm, vias 7 -> 8
- net /RST: track 80.7 -> 82.8 mm, vias 0 -> 2
- net +3V3: track 49.8 -> 48.1 mm
- net /IRQ: track 106.4 -> 107.3 mm
