File: t100-nanopi-duo/board/t100-nanopi-duo.kicad_pcb (KiCad board)
At the start: 2 copper layers, 30 x 100 mm, 15 parts, among them J1 USB_B_Micro, J2 UART, J3 Raspberry_Pi_Zero_2_W, J4 T100-IN, J5 T100-OUT, U1 CH330N

Commit message: WIP
Parts:
- removed J3: Raspberry_Pi_Zero_2_W, Drake:Raspberry-Pi-Zero-2-W-horizontal-4-holes
- added M1: NanoPi-Duo, Drake:NanoPi-Duo, F.Cu at (125.0, 119.0)
- moved J2 26.0 mm to (121.0, 90.5)
- moved C3 8.94 mm to (121.0, 82.0), turned to 180 degrees
Routing:
- net +5V: track 49.1 -> 91.5 mm
- net /SDA: track 40.2 -> 75.3 mm, vias 1 -> 0
- net /SCL: track 42.9 -> 76.0 mm, vias 1 -> 0
- net /IRQ: track 107.3 -> 98.0 mm
- net /MY_RXD: track 56.2 -> 65.0 mm, vias 1 -> 2
- net /MY_TXD: track 53.0 -> 59.0 mm, vias 1 -> 0
- net /RST: track 82.8 -> 80.7 mm, vias 2 -> 0
Other:
- board text added: "T100-NANOPI DUO v2.0"
- board text removed: "T100-RASPI ZERO v2.0"
